File: x-register.kicad_sch (KiCad schematic)
At the start: 24 parts, among them U43 74HCT193, U46 74HCT193, U56 74HCT00, U7 74HCT245

Commit message: changed symbols
Parts:
- U43, U46: symbol 74xx:74LS193 -> 01_my_library:74HCT193
- U7: symbol 74xx:74HC245 -> 01_my_library:74HCT245
Changed lines of the file:
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@@
     )
   )
-  (symbol (lib_id "74xx:74HC245") (at 86.36 101.6 90) (unit 1)
+  (symbol (lib_id "01_my_library:74HCT245") (at 86.36 101.6 90) (unit 1)
     (in_bom yes) (on_board yes) (dnp no)
     (property "Reference" "U7" (at 106.68 95.25 90)
@@
       (effects (font (size 1.27 1.27)) hide)
     )
-    (property "Datasheet" "http://www.ti.com/lit/gpn/sn74HC245" (at 86.36 101.6 0)
+    (property "Datasheet" "https://www.ti.com/lit/ds/symlink/sn74hct245.pdf?ts=1702763405638&ref_url=https%253A%252F%252Fwww.google.com%252F" (at 109.22 101.6 0)
       (effects (font (size 1.27 1.27)) hide)
     )
@@
     )
   )
-  (symbol (lib_id "74xx:74LS193") (at 156.21 101.6 270) (unit 1)
-    (in_bom yes) (on_board yes) (dnp no) (fields_autoplaced)
-    (property "Reference" "U46" (at 173.99 94.6719 90)
-      (effects (font (size 1.27 1.27)))
-    )
-    (property "Value" "74HCT193" (at 173.99 97.2119 90)
-      (effects (font (size 1.27 1.27)))
-    )
-    (property "Footprint" "" (at 156.21 101.6 0)
-      (effects (font (size 1.27 1.27)) hide)
-    )
-    (property "Datasheet" "http://www.ti.com/lit/ds/symlink/sn74ls193.pdf" (at 156.21 101.6 0)
+  (symbol (lib_id "01_my_library:74HCT193") (at 154.94 101.6 270) (unit 1)
+    (in_bom yes) (on_board yes) (dnp no) (fields_autoplaced)
+    (property "Reference" "U46" (at 175.26 94.6719 90)
+      (effects (font (size 1.27 1.27)))
+    )
+    (property "Value" "74HCT193" (at 175.26 97.2119 90)
+      (effects (font (size 1.27 1.27)))
+    )
+    (property "Footprint" "" (at 154.94 101.6 0)
+      (effects (font (size 1.27 1.27)) hide)
+    )
+    (property "Datasheet" "https://www.ti.com/lit/ds/symlink/cd74hct193.pdf?HQS=dis-mous-null-mousermode-dsf-pf-null-wwe&ts=1702791971938&ref_url=https%253A%252F%252Fwww.mouser.be%252F" (at 139.7 101.6 0)
       (effects (font (size 1.27 1.27)) hide)
     )
@@
     )
   )
-  (symbol (lib_id "74xx:74LS193") (at 219.71 101.6 270) (unit 1)
-    (in_bom yes) (on_board yes) (dnp no) (fields_autoplaced)
-    (property "Reference" "U43" (at 237.49 94.6719 90)
-      (effects (font (size 1.27 1.27)))
-    )
-    (property "Value" "74HCT193" (at 237.49 97.2119 90)
-      (effects (font (size 1.27 1.27)))
-    )
-    (property "Footprint" "" (at 219.71 101.6 0)
-      (effects (font (size 1.27 1.27)) hide)
-    )
-    (property "Datasheet" "http://www.ti.com/lit/ds/symlink/sn74ls193.pdf" (at 219.71 101.6 0)
-      (effects (font (size 1.27 1.27)) hide)
-    )
+  (symbol (lib_id "01_my_library:74HCT193") (at 218.44 101.6 270) (unit 1)
+    (in_bom yes) (on_board yes) (dnp no) (fields_autoplaced)
+    (property "Reference" "U43" (at 238.76 94.6719 90)
+      (effects (font (size 1.27 1.27)))
+    )
+    (property "Value" "74HCT193" (at 238.76 97.2119 90)
+      (effects (font (size 1.27 1.27)))
+    )
+    (property "Footprint" "" (at 218.44 101.6 0)
+      (effects (font (size 1.27 1.27)) hide)
+    )
+    (property "Datasheet" "https://www.ti.com/lit/ds/symlink/cd74hct193.pdf?HQS=dis-mous-null-mousermode-dsf-pf-null-wwe&ts=1702791971938&ref_url=https%253A%252F%252Fwww.mouser.be%252F" (at 203.2 101.6 0)
+      (effects (font (size 1.27 1.27)) hide)
+    )

Commit message: some cleanup
Parts:
- renumbered U46 to U58, U43 to U59
Changed lines of the file:
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@@
         )
         (path "/100bb8d1-c3d6-4e1f-87b6-72e4e187243c/54bf2e20-7ca1-4029-bb63-3da9aa82cef3"
-          (reference "#PWR0174") (unit 1)
+          (reference "#PWR0228") (unit 1)
         )
       )
@@
         )
         (path "/100bb8d1-c3d6-4e1f-87b6-72e4e187243c/54bf2e20-7ca1-4029-bb63-3da9aa82cef3"
-          (reference "R158") (unit 1)
+          (reference "R159") (unit 1)
         )
       )
@@
         )
         (path "/100bb8d1-c3d6-4e1f-87b6-72e4e187243c/54bf2e20-7ca1-4029-bb63-3da9aa82cef3"
-          (reference "R152") (unit 1)
+          (reference "R153") (unit 1)
         )
       )
@@
         )
         (path "/100bb8d1-c3d6-4e1f-87b6-72e4e187243c/54bf2e20-7ca1-4029-bb63-3da9aa82cef3"
-          (reference "#PWR0240") (unit 1)
+          (reference "#PWR0227") (unit 1)
         )
       )
@@
         )
         (path "/100bb8d1-c3d6-4e1f-87b6-72e4e187243c/54bf2e20-7ca1-4029-bb63-3da9aa82cef3"
-          (reference "D110") (unit 1)
+          (reference "D111") (unit 1)
         )
       )
@@
         )
         (path "/100bb8d1-c3d6-4e1f-87b6-72e4e187243c/54bf2e20-7ca1-4029-bb63-3da9aa82cef3"
-          (reference "D111") (unit 1)
+          (reference "D112") (unit 1)
         )
       )
@@
         )
         (path "/100bb8d1-c3d6-4e1f-87b6-72e4e187243c/54bf2e20-7ca1-4029-bb63-3da9aa82cef3"
-          (reference "#PWR0221") (unit 1)
+          (reference "#PWR0234") (unit 1)
         )
       )
@@
         )
         (path "/100bb8d1-c3d6-4e1f-87b6-72e4e187243c/54bf2e20-7ca1-4029-bb63-3da9aa82cef3"
-          (reference "#PWR0224") (unit 1)
+          (reference "#PWR0233") (unit 1)
         )
       )
@@
         )
         (path "/100bb8d1-c3d6-4e1f-87b6-72e4e187243c/54bf2e20-7ca1-4029-bb63-3da9aa82cef3"
-          (reference "#PWR0175") (unit 1)
+          (reference "#PWR0231") (unit 1)
         )
       )
@@
         )
         (path "/100bb8d1-c3d6-4e1f-87b6-72e4e187243c/54bf2e20-7ca1-4029-bb63-3da9aa82cef3"
-          (reference "U55") (unit 1)
+          (reference "U57") (unit 1)
         )
       )
@@
         )
         (path "/100bb8d1-c3d6-4e1f-87b6-72e4e187243c/54bf2e20-7ca1-4029-bb63-3da9aa82cef3"
-          (reference "C63") (unit 1)
+          (reference "C65") (unit 1)
         )
       )
@@
         )
         (path "/100bb8d1-c3d6-4e1f-87b6-72e4e187243c/54bf2e20-7ca1-4029-bb63-3da9aa82cef3"
-          (reference "D107") (unit 1)
+          (reference "D108") (unit 1)
         )
       )
@@
         )
         (path "/100bb8d1-c3d6-4e1f-87b6-72e4e187243c/54bf2e20-7ca1-4029-bb63-3da9aa82cef3"
-          (reference "#PWR0169") (unit 1)
+          (reference "#PWR0235") (unit 1)
         )
       )
@@
         )
         (path "/100bb8d1-c3d6-4e1f-87b6-72e4e187243c/54bf2e20-7ca1-4029-bb63-3da9aa82cef3"
-          (reference "R156") (unit 1)
+          (reference "R157") (unit 1)
         )
       )
@@
         )
         (path "/100bb8d1-c3d6-4e1f-87b6-72e4e187243c/54bf2e20-7ca1-4029-bb63-3da9aa82cef3"
-          (reference "#PWR0239") (unit 1)
+          (reference "#PWR0226") (unit 1)
         )
       )
@@
         )
         (path "/100bb8d1-c3d6-4e1f-87b6-72e4e187243c/54bf2e20-7ca1-4029-bb63-3da9aa82cef3"
-          (reference "D112") (unit 1)
+          (reference "D113") (unit 1)
         )
       )
@@
         )
         (path "/100bb8d1-c3d6-4e1f-87b6-72e4e187243c/54bf2e20-7ca1-4029-bb63-3da9aa82cef3"
-          (reference "R154") (unit 1)
+          (reference "R155") (unit 1)
         )
       )
@@
         )
         (path "/100bb8d1-c3d6-4e1f-87b6-72e4e187243c/54bf2e20-7ca1-4029-bb63-3da9aa82cef3"
-          (reference "D109") (unit 1)
+          (reference "D110") (unit 1)
         )
       )
@@
         )
         (path "/100bb8d1-c3d6-4e1f-87b6-72e4e187243c/54bf2e20-7ca1-4029-bb63-3da9aa82cef3"
-          (reference "#PWR0225") (unit 1)
+          (reference "#PWR0238") (unit 1)
         )
       )
@@
         )
         (path "/100bb8d1-c3d6-4e1f-87b6-72e4e187243c/54bf2e20-7ca1-4029-bb63-3da9aa82cef3"
-          (reference "#PWR0238") (unit 1)
+          (reference "#PWR0225") (unit 1)
         )
       )
@@
         )
         (path "/100bb8d1-c3d6-4e1f-87b6-72e4e187243c/54bf2e20-7ca1-4029-bb63-3da9aa82cef3"
-          (reference "#PWR0223") (unit 1)
+          (reference "#PWR0232") (unit 1)
         )
       )
@@
         )
         (path "/100bb8d1-c3d6-4e1f-87b6-72e4e187243c/54bf2e20-7ca1-4029-bb63-3da9aa82cef3"
-          (reference "D114") (unit 1)
+          (reference "D115") (unit 1)
         )
       )
@@
   (symbol (lib_id "01_my_library:74HCT193") (at 154.94 101.6 270) (unit 1)
     (in_bom yes) (on_board yes) (dnp no) (fields_autoplaced)
-    (property "Reference" "U46" (at 175.26 94.6719 90)
+    (property "Reference" "U58" (at 175.26 94.6719 90)
       (effects (font (size 1.27 1.27)))
     )
@@
       (project "8-bit-cpu"
         (path "/100bb8d1-c3d6-4e1f-87b6-72e4e187243c/54bf2e20-7ca1-4029-bb63-3da9aa82cef3"
-          (reference "U46") (unit 1)
+          (reference "U58") (unit 1)
         )
       )
@@
         )
         (path "/100bb8d1-c3d6-4e1f-87b6-72e4e187243c/54bf2e20-7ca1-4029-bb63-3da9aa82cef3"
-          (reference "R155") (unit 1)
+          (reference "R156") (unit 1)
         )
       )
@@
         )
         (path "/100bb8d1-c3d6-4e1f-87b6-72e4e187243c/54bf2e20-7ca1-4029-bb63-3da9aa82cef3"
-          (reference "#PWR0171") (unit 1)
+          (reference "#PWR0230") (unit 1)
         )
       )
@@
         )
         (path "/100bb8d1-c3d6-4e1f-87b6-72e4e187243c/54bf2e20-7ca1-4029-bb63-3da9aa82cef3"
-          (reference "R151") (unit 1)
+          (reference "R152") (unit 1)
         )
       )
@@
         )
         (path "/100bb8d1-c3d6-4e1f-87b6-72e4e187243c/54bf2e20-7ca1-4029-bb63-3da9aa82cef3"
-          (reference "C49") (unit 1)
+          (reference "C66") (unit 1)
         )
       )
@@
         )
         (path "/100bb8d1-c3d6-4e1f-87b6-72e4e187243c/54bf2e20-7ca1-4029-bb63-3da9aa82cef3"
-          (reference "#PWR0168") (unit 1)
+          (reference "#PWR0229") (unit 1)
         )
       )
@@
         )
         (path "/100bb8d1-c3d6-4e1f-87b6-72e4e187243c/54bf2e20-7ca1-4029-bb63-3da9aa82cef3"
-          (reference "#PWR0222") (unit 1)
+          (reference "#PWR0237") (unit 1)
         )
       )
@@
         )
         (path "/100bb8d1-c3d6-4e1f-87b6-72e4e187243c/54bf2e20-7ca1-4029-bb63-3da9aa82cef3"
-          (reference "C67") (unit 1)
+          (reference "C64") (unit 1)
         )
       )
@@
         )
         (path "/100bb8d1-c3d6-4e1f-87b6-72e4e187243c/54bf2e20-7ca1-4029-bb63-3da9aa82cef3"
-          (reference "#PWR0172") (unit 1)
+          (reference "#PWR0236") (unit 1)
         )
       )
@@
         )
         (path "/100bb8d1-c3d6-4e1f-87b6-72e4e187243c/54bf2e20-7ca1-4029-bb63-3da9aa82cef3"
-          (reference "D108") (unit 1)
+          (reference "D109") (unit 1)
         )
       )
@@
   (symbol (lib_id "01_my_library:74HCT193") (at 218.44 101.6 270) (unit 1)
     (in_bom yes) (on_board yes) (dnp no) (fields_autoplaced)
-    (property "Reference" "U43" (at 238.76 94.6719 90)
+    (property "Reference" "U59" (at 238.76 94.6719 90)
       (effects (font (size 1.27 1.27)))
     )
@@
       (project "8-bit-cpu"
         (path "/100bb8d1-c3d6-4e1f-87b6-72e4e187243c/54bf2e20-7ca1-4029-bb63-3da9aa82cef3"
-          (reference "U43") (unit 1)
+          (reference "U59") (unit 1)
         )
       )
@@
         )
         (path "/100bb8d1-c3d6-4e1f-87b6-72e4e187243c/54bf2e20-7ca1-4029-bb63-3da9aa82cef3"
-          (reference "R157") (unit 1)
+          (reference "R158") (unit 1)
         )
       )
@@
         )
         (path "/100bb8d1-c3d6-4e1f-87b6-72e4e187243c/54bf2e20-7ca1-4029-bb63-3da9aa82cef3"
-          (reference "D113") (unit 1)
+          (reference "D114") (unit 1)
         )
       )
@@
         )
         (path "/100bb8d1-c3d6-4e1f-87b6-72e4e187243c/54bf2e20-7ca1-4029-bb63-3da9aa82cef3"
-          (reference "R153") (unit 1)
+          (reference "R154") (unit 1)
         )
       )
@@
         )
         (path "/100bb8d1-c3d6-4e1f-87b6-72e4e187243c/54bf2e20-7ca1-4029-bb63-3da9aa82cef3"
-          (reference "C50") (unit 1)
-        )
-      )
+          (reference "C67") (unit 1)
+        )
+      )

Commit message: add arduino headers for programming
Parts:
- U56: footprint (none) -> Package_DIP:DIP-14_W7.62mm
- U58, U59: footprint (none) -> Package_DIP:DIP-16_W7.62mm
Changed lines of the file:
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@@
       (effects (font (size 1.27 1.27)) (justify left))
     )
-    (property "Footprint" "" (at 264.16 41.91 0)
+    (property "Footprint" "Package_DIP:DIP-14_W7.62mm" (at 264.16 41.91 0)
       (effects (font (size 1.27 1.27)) hide)
     )
@@
       (effects (font (size 1.27 1.27)))
     )
-    (property "Footprint" "" (at 91.44 24.13 0)
+    (property "Footprint" "Package_DIP:DIP-14_W7.62mm" (at 91.44 24.13 0)
       (effects (font (size 1.27 1.27)) hide)
     )
@@
       (effects (font (size 1.27 1.27)))
     )
-    (property "Footprint" "" (at 154.94 101.6 0)
+    (property "Footprint" "Package_DIP:DIP-16_W7.62mm" (at 154.94 101.6 0)
       (effects (font (size 1.27 1.27)) hide)
     )
@@
       (effects (font (size 1.27 1.27)))
     )
-    (property "Footprint" "" (at 218.44 101.6 0)
+    (property "Footprint" "Package_DIP:DIP-16_W7.62mm" (at 218.44 101.6 0)
       (effects (font (size 1.27 1.27)) hide)
     )
@@
       (effects (font (size 1.27 1.27)))
     )
-    (property "Footprint" "" (at 91.44 39.37 0)
-      (effects (font (size 1.27 1.27)) hide)
-    )
+    (property "Footprint" "Package_DIP:DIP-14_W7.62mm" (at 91.44 39.37 0)
+      (effects (font (size 1.27 1.27)) hide)
+    )

Commit message: trying to solve issues
Parts:
- added C9: 100n, 01_my_library:C_Disc_D4.0mm_W2.6mm_P2.50mm, symbol Device:C
- added U59: 74HCT00, symbol 74xx:74HCT00
- renumbered U56 to U58, U58 to U61, U59 to U62
Connections:
- net +5V: now also C9.1, U59.14 (VCC)
- net CLOCK: now also U59.1
- net GND: now also C9.2, U59.10, U59.12, U59.13, U59.4, U59.5, U59.7 (GND), U59.9
- net ~{X_INPUT} renamed X_INPUT_TRG
- net X_INPUT_TRG: now also U59.3
- new net X_INPUT: U59.2
- no-connect marks 2 -> 5
Other:
- note added: "Logic gates power"
- note added: "Unused gates"
- note removed: "Logic gates power (Other 2 gates are on Stack)"
- moved on the sheet: C1, D13, D14, D15, D16, D17, D18, D19, D20, R27, R28, R29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
