File: x-register.kicad_sch (KiCad schematic)
At the start: 26 parts, among them U58 74HCT00, U59 74HCT00, U61 74HCT193, U62 74HCT193, U7 74HCT245

Commit message: regenerated BOM
Parts:
- U59: footprint (none) -> Package_DIP:DIP-14_W7.62mm
Changed lines of the file:
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@@
       (effects (font (size 1.27 1.27)))
     )
-    (property "Footprint" "" (at 229.87 152.4 0)
+    (property "Footprint" "Package_DIP:DIP-14_W7.62mm" (at 229.87 152.4 0)
       (effects (font (size 1.27 1.27)) hide)
     )
@@
       (effects (font (size 1.27 1.27)))
     )
-    (property "Footprint" "" (at 251.46 152.4 0)
+    (property "Footprint" "Package_DIP:DIP-14_W7.62mm" (at 251.46 152.4 0)
       (effects (font (size 1.27 1.27)) hide)
     )
@@
       (effects (font (size 1.27 1.27)))
     )
-    (property "Footprint" "" (at 271.78 152.4 0)
+    (property "Footprint" "Package_DIP:DIP-14_W7.62mm" (at 271.78 152.4 0)
       (effects (font (size 1.27 1.27)) hide)
     )
@@
       (effects (font (size 1.27 1.27)))
     )
-    (property "Footprint" "" (at 219.71 72.39 0)
+    (property "Footprint" "Package_DIP:DIP-14_W7.62mm" (at 219.71 72.39 0)
       (effects (font (size 1.27 1.27)) hide)
     )
@@
       (effects (font (size 1.27 1.27)) (justify left))
     )
-    (property "Footprint" "" (at 234.95 41.91 0)
-      (effects (font (size 1.27 1.27)) hide)
-    )
+    (property "Footprint" "Package_DIP:DIP-14_W7.62mm" (at 234.95 41.91 0)
+      (effects (font (size 1.27 1.27)) hide)
+    )

Commit message: readme
Parts:
- added C13: 10n, 01_my_library:C_Disc_D4.0mm_W2.6mm_P2.50mm, symbol Device:C
Connections:
- net GND: now also C13.2
- net RESET: now also C13.1
Changed lines of the file:
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@@
   (junction (at 220.98 101.6) (diameter 0) (color 0 0 0 0)
+  )
+  (junction (at 181.61 72.39) (diameter 0) (color 255 0 0 1)
   )
   (junction (at 242.57 154.94) (diameter 0) (color 0 0 0 0)
@@
     (stroke (width 0) (type default))
   )
+  (wire (pts (xy 167.64 58.42) (xy 167.64 59.69))
+    (stroke (width 0) (type default) (color 255 0 0 1))
+  )
   (wire (pts (xy 191.77 86.36) (xy 191.77 88.9))
     (stroke (width 0) (type default))
@@
     (stroke (width 0) (type default) (color 0 0 255 1))
   )
+  (wire (pts (xy 181.61 58.42) (xy 167.64 58.42))
+    (stroke (width 0) (type default) (color 255 0 0 1))
+  )
   (wire (pts (xy 80.01 158.75) (xy 189.23 158.75))
     (stroke (width 0) (type default))
@@
   (wire (pts (xy 120.65 134.62) (xy 120.65 148.59))
     (stroke (width 0) (type default))
+  )
+  (wire (pts (xy 181.61 72.39) (xy 181.61 58.42))
+    (stroke (width 0) (type default) (color 255 0 0 1))
   )
   (wire (pts (xy 69.85 121.92) (xy 66.04 121.92))
@@
     )
   )
+  (symbol (lib_id "power:GND") (at 167.64 67.31 0) (unit 1)
+    (in_bom yes) (on_board yes) (dnp no) (fields_autoplaced)
+    (property "Reference" "#PWR03" (at 167.64 73.66 0)
+      (effects (font (size 1.27 1.27)) hide)
+    )
+    (property "Value" "GND" (at 167.64 72.39 0)
+      (effects (font (size 1.27 1.27)) hide)
+    )
+    (property "Footprint" "" (at 167.64 67.31 0)
+      (effects (font (size 1.27 1.27)) hide)
+    )
+    (property "Datasheet" "" (at 167.64 67.31 0)
+      (effects (font (size 1.27 1.27)) hide)
+    )
+    (pin "1")
+    (instances
+      (project "8-bit-cpu"
+        (path "/100bb8d1-c3d6-4e1f-87b6-72e4e187243c/45eb39c3-c748-461e-8330-08aae1247dee"
+          (reference "#PWR03") (unit 1)
+        )
+        (path "/100bb8d1-c3d6-4e1f-87b6-72e4e187243c/651dfbaf-e340-4976-8216-793c5a5aaa3b"
+          (reference "#PWR038") (unit 1)
+        )
+        (path "/100bb8d1-c3d6-4e1f-87b6-72e4e187243c/3568514a-e420-48fa-9fd5-7a290120765b"
+          (reference "#PWR056") (unit 1)
+        )
+        (path "/100bb8d1-c3d6-4e1f-87b6-72e4e187243c/54bf2e20-7ca1-4029-bb63-3da9aa82cef3"
+          (reference "#PWR0270") (unit 1)
+        )
+      )
+    )
+  )
   (symbol (lib_id "power:+5V") (at 88.9 110.49 0) (unit 1)
     (in_bom yes) (on_board yes) (dnp no) (fields_autoplaced)
@@
         )
       )
+    )
+  )
+  (symbol (lib_id "Device:C") (at 167.64 63.5 0) (unit 1)
+    (in_bom yes) (on_board yes) (dnp yes) (fields_autoplaced)
+    (property "Reference" "C13" (at 171.45 62.23 0)
+      (effects (font (size 1.27 1.27)) (justify left))
+    )
+    (property "Value" "10n" (at 171.45 64.77 0)
+      (effects (font (size 1.27 1.27)) (justify left))
+    )
+    (property "Footprint" "01_my_library:C_Disc_D4.0mm_W2.6mm_P2.50mm" (at 168.6052 67.31 0)
+      (effects (font (size 1.27 1.27)) hide)
+    )
+    (property "Datasheet" "~" (at 167.64 63.5 0)
+      (effects (font (size 1.27 1.27)) hide)
+    )
+    (pin "1")
+    (pin "2")
+    (instances
+      (project "8-bit-cpu"
+        (path "/100bb8d1-c3d6-4e1f-87b6-72e4e187243c/651dfbaf-e340-4976-8216-793c5a5aaa3b"
+          (reference "C13") (unit 1)
+        )
+        (path "/100bb8d1-c3d6-4e1f-87b6-72e4e187243c/54bf2e20-7ca1-4029-bb63-3da9aa82cef3"
+          (reference "C82") (unit 1)
+        )
+      )

Commit message: kicad update
Parts:
- D107: renamed from D13; footprint LED_THT:LED_D5.0mm -> 01_my_library:LED_D5.0mm
- D108: renamed from D14; footprint LED_THT:LED_D5.0mm -> 01_my_library:LED_D5.0mm
- D109: renamed from D15; footprint LED_THT:LED_D5.0mm -> 01_my_library:LED_D5.0mm
- D110: renamed from D16; footprint LED_THT:LED_D5.0mm -> 01_my_library:LED_D5.0mm
- D111: renamed from D17; footprint LED_THT:LED_D5.0mm -> 01_my_library:LED_D5.0mm
- D112: renamed from D18; footprint LED_THT:LED_D5.0mm -> 01_my_library:LED_D5.0mm
- D113: renamed from D19; footprint LED_THT:LED_D5.0mm -> 01_my_library:LED_D5.0mm
- D114: renamed from D20; footprint LED_THT:LED_D5.0mm -> 01_my_library:LED_D5.0mm
- renumbered C9 to C73, C9 to C74, C13 to C75, C1 to C76, C1 to C77, C1 to C78, R27 to R151, R28 to R152, R29 to R153, R30 to R154, R31 to R155, R32 to R156, R33 to R157, R34 to R158, U7 to U60
