File: ram-logic.kicad_sch (KiCad schematic)
At the start: 17 parts, among them SW1 Button, SW202 Programming Switch, U26 74HCT00, U31 74HCT157

Commit message: some cleanup
Parts:
- renumbered D55 to D56, R86 to R87, R87 to R88
Changed lines of the file:
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@@
         )
         (path "/100bb8d1-c3d6-4e1f-87b6-72e4e187243c/33b906b8-f63f-4a46-8ef2-4150917936b8/bcf72b05-a298-432c-8bad-dccda5c38b50"
-          (reference "#PWR0123") (unit 1)
+          (reference "#PWR0122") (unit 1)
         )
       )
@@
         )
         (path "/100bb8d1-c3d6-4e1f-87b6-72e4e187243c/33b906b8-f63f-4a46-8ef2-4150917936b8/bcf72b05-a298-432c-8bad-dccda5c38b50"
-          (reference "#PWR0124") (unit 1)
+          (reference "#PWR0123") (unit 1)
         )
       )
@@
   (symbol (lib_id "Device:D_Schottky") (at 43.18 165.1 180) (unit 1)
     (in_bom yes) (on_board yes) (dnp no)
-    (property "Reference" "D55" (at 43.18 168.91 0)
+    (property "Reference" "D56" (at 43.18 168.91 0)
       (effects (font (size 1.27 1.27)))
     )
@@
       (project "8-bit-cpu"
         (path "/100bb8d1-c3d6-4e1f-87b6-72e4e187243c/33b906b8-f63f-4a46-8ef2-4150917936b8/bcf72b05-a298-432c-8bad-dccda5c38b50"
-          (reference "D55") (unit 1)
+          (reference "D56") (unit 1)
         )
       )
@@
         )
         (path "/100bb8d1-c3d6-4e1f-87b6-72e4e187243c/33b906b8-f63f-4a46-8ef2-4150917936b8/bcf72b05-a298-432c-8bad-dccda5c38b50"
-          (reference "D53") (unit 1)
+          (reference "D54") (unit 1)
         )
       )
@@
         )
         (path "/100bb8d1-c3d6-4e1f-87b6-72e4e187243c/33b906b8-f63f-4a46-8ef2-4150917936b8/bcf72b05-a298-432c-8bad-dccda5c38b50"
-          (reference "R84") (unit 1)
+          (reference "R85") (unit 1)
         )
       )
@@
         )
         (path "/100bb8d1-c3d6-4e1f-87b6-72e4e187243c/33b906b8-f63f-4a46-8ef2-4150917936b8/bcf72b05-a298-432c-8bad-dccda5c38b50"
-          (reference "R85") (unit 1)
+          (reference "R86") (unit 1)
         )
       )
@@
         )
         (path "/100bb8d1-c3d6-4e1f-87b6-72e4e187243c/33b906b8-f63f-4a46-8ef2-4150917936b8/bcf72b05-a298-432c-8bad-dccda5c38b50"
-          (reference "#PWR0122") (unit 1)
+          (reference "#PWR0121") (unit 1)
         )
       )
@@
         )
         (path "/100bb8d1-c3d6-4e1f-87b6-72e4e187243c/33b906b8-f63f-4a46-8ef2-4150917936b8/bcf72b05-a298-432c-8bad-dccda5c38b50"
-          (reference "#PWR0116") (unit 1)
+          (reference "#PWR0115") (unit 1)
         )
       )
@@
         )
         (path "/100bb8d1-c3d6-4e1f-87b6-72e4e187243c/33b906b8-f63f-4a46-8ef2-4150917936b8/bcf72b05-a298-432c-8bad-dccda5c38b50"
-          (reference "R83") (unit 1)
+          (reference "R84") (unit 1)
         )
       )
@@
         )
         (path "/100bb8d1-c3d6-4e1f-87b6-72e4e187243c/33b906b8-f63f-4a46-8ef2-4150917936b8/bcf72b05-a298-432c-8bad-dccda5c38b50"
-          (reference "#PWR0118") (unit 1)
+          (reference "#PWR0117") (unit 1)
         )
       )
@@
         )
         (path "/100bb8d1-c3d6-4e1f-87b6-72e4e187243c/33b906b8-f63f-4a46-8ef2-4150917936b8/bcf72b05-a298-432c-8bad-dccda5c38b50"
-          (reference "#PWR0120") (unit 1)
+          (reference "#PWR0119") (unit 1)
         )
       )
@@
         )
         (path "/100bb8d1-c3d6-4e1f-87b6-72e4e187243c/33b906b8-f63f-4a46-8ef2-4150917936b8/bcf72b05-a298-432c-8bad-dccda5c38b50"
-          (reference "#PWR0119") (unit 1)
+          (reference "#PWR0118") (unit 1)
         )
       )
@@
         )
         (path "/100bb8d1-c3d6-4e1f-87b6-72e4e187243c/33b906b8-f63f-4a46-8ef2-4150917936b8/bcf72b05-a298-432c-8bad-dccda5c38b50"
-          (reference "#PWR0126") (unit 1)
+          (reference "#PWR0125") (unit 1)
         )
       )
@@
   (symbol (lib_id "Device:R") (at 109.22 149.86 0) (unit 1)
     (in_bom yes) (on_board yes) (dnp no) (fields_autoplaced)
-    (property "Reference" "R86" (at 111.76 148.59 0)
+    (property "Reference" "R87" (at 111.76 148.59 0)
       (effects (font (size 1.27 1.27)) (justify left))
     )
@@
       (project "8-bit-cpu"
         (path "/100bb8d1-c3d6-4e1f-87b6-72e4e187243c/33b906b8-f63f-4a46-8ef2-4150917936b8/bcf72b05-a298-432c-8bad-dccda5c38b50"
-          (reference "R86") (unit 1)
+          (reference "R87") (unit 1)
         )
       )
@@
         )
         (path "/100bb8d1-c3d6-4e1f-87b6-72e4e187243c/33b906b8-f63f-4a46-8ef2-4150917936b8/bcf72b05-a298-432c-8bad-dccda5c38b50"
-          (reference "#PWR0125") (unit 1)
+          (reference "#PWR0124") (unit 1)
         )
       )
@@
         )
         (path "/100bb8d1-c3d6-4e1f-87b6-72e4e187243c/33b906b8-f63f-4a46-8ef2-4150917936b8/bcf72b05-a298-432c-8bad-dccda5c38b50"
-          (reference "#PWR0121") (unit 1)
+          (reference "#PWR0120") (unit 1)
         )
       )
@@
         )
         (path "/100bb8d1-c3d6-4e1f-87b6-72e4e187243c/33b906b8-f63f-4a46-8ef2-4150917936b8/bcf72b05-a298-432c-8bad-dccda5c38b50"
-          (reference "D54") (unit 1)
+          (reference "D55") (unit 1)
         )
       )
@@
   (symbol (lib_id "Device:R") (at 62.23 177.8 0) (unit 1)
     (in_bom yes) (on_board yes) (dnp no) (fields_autoplaced)
-    (property "Reference" "R87" (at 64.77 176.53 0)
+    (property "Reference" "R88" (at 64.77 176.53 0)
       (effects (font (size 1.27 1.27)) (justify left))
     )
@@
       (project "8-bit-cpu"
         (path "/100bb8d1-c3d6-4e1f-87b6-72e4e187243c/33b906b8-f63f-4a46-8ef2-4150917936b8/bcf72b05-a298-432c-8bad-dccda5c38b50"
-          (reference "R87") (unit 1)
+          (reference "R88") (unit 1)
         )
       )
@@
         )
         (path "/100bb8d1-c3d6-4e1f-87b6-72e4e187243c/33b906b8-f63f-4a46-8ef2-4150917936b8/bcf72b05-a298-432c-8bad-dccda5c38b50"
-          (reference "#PWR0115") (unit 1)
+          (reference "#PWR0114") (unit 1)
         )
       )
@@
         )
         (path "/100bb8d1-c3d6-4e1f-87b6-72e4e187243c/33b906b8-f63f-4a46-8ef2-4150917936b8/bcf72b05-a298-432c-8bad-dccda5c38b50"
-          (reference "#PWR0117") (unit 1)
-        )
-      )
+          (reference "#PWR0116") (unit 1)
+        )
+      )

Commit message: add arduino headers for programming
Parts:
- added J3: Arduino_Programming_Trigger_Header, Connector_PinSocket_2.54mm:PinSocket_1x02_P2.54mm_Vertical, symbol Connector:Conn_01x02_Socket
Connections:
- net GND: now also J3.1 (Pin_1)
- net at R87.1, SW1.2, U31.3 (1B): now also J3.2 (Pin_2)
Changed lines of the file:
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@@
   (junction (at 116.84 154.94) (diameter 0) (color 0 0 0 0)
   )
+  (junction (at 99.06 129.54) (diameter 0) (color 0 0 0 0)
+  )
   (junction (at 123.19 135.89) (diameter 0) (color 0 0 0 0)
   )
@@
   )
   (junction (at 50.8 160.02) (diameter 0) (color 255 0 0 1)
+  )
+  (junction (at 80.01 142.24) (diameter 0) (color 0 0 0 0)
   )
   (junction (at 223.52 113.03) (diameter 0) (color 0 0 0 0)
@@
     (stroke (width 0) (type default) (color 255 0 0 1))
   )
+  (wire (pts (xy 74.93 127) (xy 80.01 127))
+    (stroke (width 0) (type default))
+  )
+  (wire (pts (xy 74.93 129.54) (xy 99.06 129.54))
+    (stroke (width 0) (type default))
+  )
   (wire (pts (xy 116.84 154.94) (xy 123.19 154.94))
     (stroke (width 0) (type default))
@@
     (stroke (width 0) (type default))
   )
+  (wire (pts (xy 80.01 127) (xy 80.01 142.24))
+    (stroke (width 0) (type default))
+  )
   (wire (pts (xy 106.68 106.68) (xy 93.98 106.68))
     (stroke (width 0) (type default))
@@
     (stroke (width 0) (type default))
   )
+  (wire (pts (xy 80.01 142.24) (xy 109.22 142.24))
+    (stroke (width 0) (type default))
+  )
   (wire (pts (xy 76.2 38.1) (xy 76.2 39.37))
     (stroke (width 0) (type default))
@@
     (stroke (width 0) (type default))
   )
-  (wire (pts (xy 73.66 142.24) (xy 109.22 142.24))
+  (wire (pts (xy 73.66 142.24) (xy 80.01 142.24))
     (stroke (width 0) (type default))
   )
@@
         )
       )
+    )
+  )
+  (symbol (lib_id "Connector:Conn_01x02_Socket") (at 69.85 129.54 180) (unit 1)
+    (in_bom yes) (on_board yes) (dnp no)
+    (property "Reference" "J3" (at 69.85 120.65 0)
+      (effects (font (size 1.27 1.27)))
+    )
+    (property "Value" "Arduino_Programming_Trigger_Header" (at 69.85 123.19 0)
+      (effects (font (size 1.27 1.27)))
+    )
+    (property "Footprint" "Connector_PinSocket_2.54mm:PinSocket_1x02_P2.54mm_Vertical" (at 69.85 129.54 0)
+      (effects (font (size 1.27 1.27)) hide)
+    )
+    (property "Datasheet" "~" (at 69.85 129.54 0)
+      (effects (font (size 1.27 1.27)) hide)
+    )
+    (pin "2")
+    (pin "1")
+    (instances
+      (project "8-bit-cpu"
+        (path "/100bb8d1-c3d6-4e1f-87b6-72e4e187243c/33b906b8-f63f-4a46-8ef2-4150917936b8/bcf72b05-a298-432c-8bad-dccda5c38b50"
+          (reference "J3") (unit 1)
+        )
+      )

Commit message: it kinda works
Parts:
- removed C1: 10n, 01_my_library:C_Disc_D4.0mm_W2.6mm_P2.50mm, symbol Device:C
- removed D56: D_Schottky, Diode_THT:D_DO-41_SOD81_P7.62mm_Horizontal, symbol Device:D_Schottky
- removed R88: 10k, Resistor_THT:R_Axial_DIN0204_L3.6mm_D1.6mm_P7.62mm_Horizontal, symbol Device:R
Connections:
- net CLOCK: now also U26.2
Changed lines of the file:
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@@
   (junction (at 223.52 113.03) (diameter 0) (color 0 0 0 0)
-  )
-  (junction (at 62.23 165.1) (diameter 0) (color 0 0 0 0)
   )
   (junction (at 109.22 142.24) (diameter 0) (color 0 0 0 0)
@@
     (stroke (width 0) (type default) (color 255 0 0 1))
   )
-  (wire (pts (xy 59.69 165.1) (xy 62.23 165.1))
-    (stroke (width 0) (type default))
-  )
   (wire (pts (xy 92.71 58.42) (xy 92.71 57.15))
     (stroke (width 0) (type default))
@@
     (stroke (width 0) (type default))
   )
-  (wire (pts (xy 62.23 165.1) (xy 63.5 165.1))
-    (stroke (width 0) (type default))
-  )
   (wire (pts (xy 93.98 106.68) (xy 93.98 109.22))
     (stroke (width 0) (type default))
@@
     (stroke (width 0) (type default))
   )
-  (wire (pts (xy 46.99 165.1) (xy 52.07 165.1))
-    (stroke (width 0) (type default))
-  )
   (wire (pts (xy 63.5 142.24) (xy 58.42 142.24))
     (stroke (width 0) (type default))
@@
     (stroke (width 0) (type default))
   )
-  (wire (pts (xy 33.02 165.1) (xy 39.37 165.1))
+  (wire (pts (xy 33.02 165.1) (xy 63.5 165.1))
     (stroke (width 0) (type default) (color 255 0 0 1))
   )
@@
   )
   (wire (pts (xy 123.19 135.89) (xy 123.19 154.94))
-    (stroke (width 0) (type default))
-  )
-  (wire (pts (xy 62.23 165.1) (xy 62.23 173.99))
     (stroke (width 0) (type default))
   )
@@
     )
   )
-  (symbol (lib_id "Device:D_Schottky") (at 43.18 165.1 180) (unit 1)
-    (in_bom yes) (on_board yes) (dnp no)
-    (property "Reference" "D56" (at 43.18 168.91 0)
-      (effects (font (size 1.27 1.27)))
-    )
-    (property "Value" "D_Schottky" (at 43.18 171.45 0)
-      (effects (font (size 1.27 1.27)))
-    )
-    (property "Footprint" "Diode_THT:D_DO-41_SOD81_P7.62mm_Horizontal" (at 43.18 165.1 0)
-      (effects (font (size 1.27 1.27)) hide)
-    )
-    (property "Datasheet" "~" (at 43.18 165.1 0)
-      (effects (font (size 1.27 1.27)) hide)
-    )
-    (pin "1")
-    (pin "2")
-    (instances
-      (project "8-bit-cpu"
-        (path "/100bb8d1-c3d6-4e1f-87b6-72e4e187243c/33b906b8-f63f-4a46-8ef2-4150917936b8/bcf72b05-a298-432c-8bad-dccda5c38b50"
-          (reference "D56") (unit 1)
-        )
-      )
-    )
-  )
   (symbol (lib_id "Device:LED") (at 99.06 36.83 0) (mirror y) (unit 1)
     (in_bom yes) (on_board yes) (dnp no)
@@
     )
   )
-  (symbol (lib_id "Device:C") (at 55.88 165.1 90) (unit 1)
-    (in_bom yes) (on_board yes) (dnp no)
-    (property "Reference" "C1" (at 57.15 168.91 90)
-      (effects (font (size 1.27 1.27)) (justify left))
-    )
-    (property "Value" "10n" (at 57.15 171.45 90)
-      (effects (font (size 1.27 1.27)) (justify left))
-    )
-    (property "Footprint" "01_my_library:C_Disc_D4.0mm_W2.6mm_P2.50mm" (at 59.69 164.1348 0)
-      (effects (font (size 1.27 1.27)) hide)
-    )
-    (property "Datasheet" "~" (at 55.88 165.1 0)
-      (effects (font (size 1.27 1.27)) hide)
-    )
-    (pin "2")
-    (pin "1")
-    (instances
-      (project "8-bit-cpu"
-        (path "/100bb8d1-c3d6-4e1f-87b6-72e4e187243c/45eb39c3-c748-461e-8330-08aae1247dee"
-          (reference "C1") (unit 1)
-        )
-        (path "/100bb8d1-c3d6-4e1f-87b6-72e4e187243c/651dfbaf-e340-4976-8216-793c5a5aaa3b"
-          (reference "C12") (unit 1)
-        )
-        (path "/100bb8d1-c3d6-4e1f-87b6-72e4e187243c/3568514a-e420-48fa-9fd5-7a290120765b"
-          (reference "C15") (unit 1)
-        )
-        (path "/100bb8d1-c3d6-4e1f-87b6-72e4e187243c/d6cd2240-d749-4685-b332-02e9e1af29c5"
-          (reference "C18") (unit 1)
-        )
-        (path "/100bb8d1-c3d6-4e1f-87b6-72e4e187243c/33b906b8-f63f-4a46-8ef2-4150917936b8"
-          (reference "C?") (unit 1)
-        )
-        (path "/100bb8d1-c3d6-4e1f-87b6-72e4e187243c/33b906b8-f63f-4a46-8ef2-4150917936b8/fa8c33ec-4897-42d8-b555-184d6239a177"
-          (reference "C42") (unit 1)
-        )
-        (path "/100bb8d1-c3d6-4e1f-87b6-72e4e187243c/33b906b8-f63f-4a46-8ef2-4150917936b8/bcf72b05-a298-432c-8bad-dccda5c38b50"
-          (reference "C37") (unit 1)
-        )
-      )
-    )
-  )
   (symbol (lib_id "Device:R") (at 113.03 48.26 0) (mirror y) (unit 1)
     (in_bom yes) (on_board yes) (dnp no) (fields_autoplaced)
@@
     )
   )
-  (symbol (lib_id "power:GND") (at 62.23 181.61 0) (unit 1)
-    (in_bom yes) (on_board yes) (dnp no) (fields_autoplaced)
-    (property "Reference" "#PWR03" (at 62.23 187.96 0)
-      (effects (font (size 1.27 1.27)) hide)
-    )
-    (property "Value" "GND" (at 62.23 186.69 0)
-      (effects (font (size 1.27 1.27)) hide)
-    )
-    (property "Footprint" "" (at 62.23 181.61 0)
-      (effects (font (size 1.27 1.27)) hide)
-    )
-    (property "Datasheet" "" (at 62.23 181.61 0)
-      (effects (font (size 1.27 1.27)) hide)
-    )
-    (pin "1")
-    (instances
-      (project "8-bit-cpu"
-        (path "/100bb8d1-c3d6-4e1f-87b6-72e4e187243c/45eb39c3-c748-461e-8330-08aae1247dee"
-          (reference "#PWR03") (unit 1)
-        )
-        (path "/100bb8d1-c3d6-4e1f-87b6-72e4e187243c/651dfbaf-e340-4976-8216-793c5a5aaa3b"
-          (reference "#PWR039") (unit 1)
-        )
-        (path "/100bb8d1-c3d6-4e1f-87b6-72e4e187243c/3568514a-e420-48fa-9fd5-7a290120765b"
-          (reference "#PWR047") (unit 1)
-        )
-        (path "/100bb8d1-c3d6-4e1f-87b6-72e4e187243c/d6cd2240-d749-4685-b332-02e9e1af29c5"
-          (reference "#PWR058") (unit 1)
-        )
-        (path "/100bb8d1-c3d6-4e1f-87b6-72e4e187243c/33b906b8-f63f-4a46-8ef2-4150917936b8"
-          (reference "#PWR?") (unit 1)
-        )
-        (path "/100bb8d1-c3d6-4e1f-87b6-72e4e187243c/33b906b8-f63f-4a46-8ef2-4150917936b8/fa8c33ec-4897-42d8-b555-184d6239a177"
-          (reference "#PWR0148") (unit 1)
-        )
-        (path "/100bb8d1-c3d6-4e1f-87b6-72e4e187243c/33b906b8-f63f-4a46-8ef2-4150917936b8/bcf72b05-a298-432c-8bad-dccda5c38b50"
-          (reference "#PWR0128") (unit 1)
-        )
-      )
-    )
-  )
   (symbol (lib_id "Device:R") (at 109.22 149.86 0) (unit 1)
     (in_bom yes) (on_board yes) (dnp no) (fields_autoplaced)
@@
         )
       )
-    )
-  )
-  (symbol (lib_id "Device:R") (at 62.23 177.8 0) (unit 1)
-    (in_bom yes) (on_board yes) (dnp no) (fields_autoplaced)
-    (property "Reference" "R88" (at 64.77 176.53 0)
-      (effects (font (size 1.27 1.27)) (justify left))
-    )
-    (property "Value" "10k" (at 64.77 179.07 0)
-      (effects (font (size 1.27 1.27)) (justify left))
-    )
-    (property "Footprint" "Resistor_THT:R_Axial_DIN0204_L3.6mm_D1.6mm_P7.62mm_Horizontal" (at 60.452 177.8 90)
-      (effects (font (size 1.27 1.27)) hide)
-    )
-    (property "Datasheet" "~" (at 62.23 177.8 0)
-      (effects (font (size 1.27 1.27)) hide)
-    )
-    (pin "2")
-    (pin "1")
-    (instances
-      (project "8-bit-cpu"
-        (path "/100bb8d1-c3d6-4e1f-87b6-72e4e187243c/33b906b8-f63f-4a46-8ef2-4150917936b8/bcf72b05-a298-432c-8bad-dccda5c38b50"
-          (reference "R88") (unit 1)
-        )
-      )
