File: ram-logic.kicad_sch (KiCad schematic)
At the start: 15 parts, among them J3 Arduino_Programming_Trigger_H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, SW1 Button, SW202 Programming Switch, U26 74HCT00, U31 74HCT157

Commit message: kicad update
Parts:
- D54: renamed from D46; footprint LED_THT:LED_D5.0mm -> 01_my_library:LED_D5.0mm
- D55: renamed from D47; footprint LED_THT:LED_D5.0mm -> 01_my_library:LED_D5.0mm
- renumbered C2 to C35, C1 to C36, C1 to C37, R74 to R84, R73 to R85, R83 to R86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
