File: 8-bit-cpu.kicad_pcb (KiCad board)
At the start: 2 copper layers, 440 parts, among them J1 Arduino_Address_Programming_H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, J2 Arduino_Data_Programming_Head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, J3 Arduino_Programming_Trigger_H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, J4 2_Complement_Header, SW1 Button, SW2 Switch, SW3 SW_DIP_x08, SW4 SW_DIP_x08, SW5 Programming Switch, SW6 Button, SW7 Button, U1 74HCT08, U10 74HCT245, U11 74HCT173, U12 74HCT173, U13 74HCT86, U14 74HCT86, U15 74HCT245, U16 74HCT283, U17 74HCT283, U18 74HCT245, U19 7130, U2 74HCT04, U20 74HCT173, U21 74HCT173, U22 74HCT157, U23 74HCT157, U24 74HCT157, U25 74HCT157, U26 74HCT00, U27 74HCT157, U28 74HCT157, U29 74HCT245, U3 74HCT32, U30 74HCT161, U31 74HCT161, U32 74HCT107, U33 74HCT139, U34 LMC555xN, U35 LTC-5723HR, U36 74HCT173, U37 AT28C64B, U38 74HCT173, U39 74HCT173, U4 LMC555xN, U40 74HCT173, U41 74HCT00, U42 74HCT173, U43 74HCT173, U44 74HCT138, U45 74HCT161, U46 74HCT04, U47 AT28C64B, U48 74HCT04, U49 AT28C64B, U5 LMC555xN, U50 74HCT04, U51 AT28C64B, U52 74HCT02, U53 74HCT08, U54 74HCT157, U55 74HCT08, U56 74HCT02, U57 74HCT173, U58 74HCT00, U59 74HCT00, U6 LMC555xN, U60 74HCT245, U61 74HCT193, U62 74HCT193, U63 74HCT245, U64 74HCT193, U65 74HCT193, U7 74HCT245, U8 74HCT173, U9 74HCT173

Commit message: readme
Parts:
- moved D8 500.4 mm to (165.0, 24.4), turned to -90 degrees
- moved D7 500.2 mm to (158.0, 24.4), turned to -90 degrees
- moved D6 496.8 mm to (151.0, 24.4), turned to -90 degrees
- moved D5 496.6 mm to (144.0, 24.4), turned to -90 degrees
- moved D4 493.7 mm to (137.0, 24.4), turned to -90 degrees
- moved D3 493.6 mm to (130.0, 24.4), turned to -90 degrees
- moved D2 491.1 mm to (123.0, 24.4), turned to -90 degrees
- moved D1 491.0 mm to (116.0, 24.4), turned to -90 degrees
- moved R8 489.2 mm to (150.8, 31.9), turned to -90 degrees
- moved R7 486.9 mm to (147.8, 31.9), turned to -90 degrees
- moved R6 484.6 mm to (144.8, 31.9), turned to -90 degrees
- moved R5 482.4 mm to (141.8, 31.9), turned to -90 degrees
- moved R4 480.2 mm to (138.8, 31.9), turned to -90 degrees
- moved R3 478.0 mm to (135.8, 31.9), turned to -90 degrees
- moved R2 475.8 mm to (132.8, 31.9), turned to -90 degrees
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