File: 8-bit-cpu.kicad_sch (KiCad schematic)
At the start: 34 parts, among them J4 Power, J5 USB_B_Micro

Commit message: kicad update
Parts:
- removed C83: 470u, Capacitor_THT:CP_Radial_D10.0mm_P5.00mm, symbol Device:C_Polarized
- removed H1, H2, H3, H4, H5, H6, H7: MountingHole, MountingHole:MountingHole_3.2mm_M3, symbol Mechanical:MountingHole
- removed J4: Power, Connector_PinSocket_2.54mm:PinSocket_1x02_P2.54mm_Vertical, symbol Connector:Conn_01x02_Socket
- removed J5: USB_B_Micro, Connector_USB:USB_Micro-B_Amphenol_10118194_Horizontal, symbol Connector:USB_B_Micro
- D1, D2, D3, D4, D5, D6, D7, D8: footprint LED_THT:LED_D5.0mm -> 01_my_library:LED_D5.0mm
Other:
- added sheet Power and Mounting (power-and-mounting.kicad_sch)
