File: alu.kicad_sch (KiCad schematic)
At the start: 26 parts, among them U13 74HCT86, U14 74HCT86, U16 74HCT283, U17 74HCT283, U7 74HCT245

Commit message: changed symbols
Parts:
- U16, U17: symbol 74xx:74LS283 -> 01_my_library:74HCT283
- U7: symbol 74xx:74HC245 -> 01_my_library:74HCT245
Changed lines of the file:
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@@
     )
   )
-  (symbol (lib_id "74xx:74LS283") (at 215.9 106.68 270) (unit 1)
-    (in_bom yes) (on_board yes) (dnp no) (fields_autoplaced)
-    (property "Reference" "U17" (at 236.22 99.7519 90)
+  (symbol (lib_id "01_my_library:74HCT283") (at 215.9 106.68 270) (unit 1)
+    (in_bom yes) (on_board yes) (dnp no) (fields_autoplaced)
+    (property "Reference" "U17" (at 237.49 99.7519 90)
       (effects (font (size 1.27 1.27)))
     )
-    (property "Value" "74HCT283" (at 236.22 102.2919 90)
+    (property "Value" "74HCT283" (at 237.49 102.2919 90)
       (effects (font (size 1.27 1.27)))
     )
@@
       (effects (font (size 1.27 1.27)) hide)
     )
-    (property "Datasheet" "http://www.ti.com/lit/gpn/sn74LS283" (at 215.9 106.68 0)
+    (property "Datasheet" "https://www.ti.com/lit/ds/symlink/cd54hct283.pdf?ts=1702794975080&ref_url=https%253A%252F%252Fwww.google.com%252F" (at 191.77 106.68 0)
       (effects (font (size 1.27 1.27)) hide)
     )
@@
     )
   )
-  (symbol (lib_id "74xx:74HC245") (at 73.66 106.68 90) (unit 1)
+  (symbol (lib_id "01_my_library:74HCT245") (at 73.66 106.68 90) (unit 1)
     (in_bom yes) (on_board yes) (dnp no)
     (property "Reference" "U7" (at 93.98 100.33 90)
@@
       (effects (font (size 1.27 1.27)) hide)
     )
-    (property "Datasheet" "http://www.ti.com/lit/gpn/sn74HC245" (at 73.66 106.68 0)
+    (property "Datasheet" "https://www.ti.com/lit/ds/symlink/sn74hct245.pdf?ts=1702763405638&ref_url=https%253A%252F%252Fwww.google.com%252F" (at 96.52 106.68 0)
       (effects (font (size 1.27 1.27)) hide)
     )
@@
     )
   )
-  (symbol (lib_id "74xx:74LS283") (at 139.7 106.68 270) (unit 1)
-    (in_bom yes) (on_board yes) (dnp no) (fields_autoplaced)
-    (property "Reference" "U16" (at 160.02 99.7519 90)
+  (symbol (lib_id "01_my_library:74HCT283") (at 139.7 106.68 270) (unit 1)
+    (in_bom yes) (on_board yes) (dnp no) (fields_autoplaced)
+    (property "Reference" "U16" (at 161.29 99.7519 90)
       (effects (font (size 1.27 1.27)))
     )
-    (property "Value" "74HCT283" (at 160.02 102.2919 90)
+    (property "Value" "74HCT283" (at 161.29 102.2919 90)
       (effects (font (size 1.27 1.27)))
     )
@@
       (effects (font (size 1.27 1.27)) hide)
     )
-    (property "Datasheet" "http://www.ti.com/lit/gpn/sn74LS283" (at 139.7 106.68 0)
-      (effects (font (size 1.27 1.27)) hide)
-    )
+    (property "Datasheet" "https://www.ti.com/lit/ds/symlink/cd54hct283.pdf?ts=1702794975080&ref_url=https%253A%252F%252Fwww.google.com%252F" (at 115.57 106.68 0)
+      (effects (font (size 1.27 1.27)) hide)
+    )

Commit message: kicad update
Parts:
- D29: renamed from D5; footprint LED_THT:LED_D5.0mm -> 01_my_library:LED_D5.0mm
- D30: renamed from D6; footprint LED_THT:LED_D5.0mm -> 01_my_library:LED_D5.0mm
- D31: renamed from D7; footprint LED_THT:LED_D5.0mm -> 01_my_library:LED_D5.0mm
- D32: renamed from D8; footprint LED_THT:LED_D5.0mm -> 01_my_library:LED_D5.0mm
- D33: renamed from D9; footprint LED_THT:LED_D5.0mm -> 01_my_library:LED_D5.0mm
- D34: renamed from D10; footprint LED_THT:LED_D5.0mm -> 01_my_library:LED_D5.0mm
- D35: renamed from D11; footprint LED_THT:LED_D5.0mm -> 01_my_library:LED_D5.0mm
- D36: renamed from D12; footprint LED_THT:LED_D5.0mm -> 01_my_library:LED_D5.0mm
- renumbered C1 to C21, C1 to C22, C1 to C23, C9 to C24, C9 to C25, R11 to R43, R12 to R44, R13 to R45, R14 to R46, R15 to R47, R16 to R48, R17 to R49, R18 to R50, U7 to U15
