File: clock.kicad_sch (KiCad schematic)
At the start: 35 parts, among them SW1 Button, SW2 Switch, U1 74HCT08, U2 74HCT04, U3 74HCT32, U4 LMC555xN, U5 LMC555xN, U6 LMC555xN

Commit message: kicad update
Parts:
- D10, D11, D12, D9: footprint LED_THT:LED_D5.0mm -> 01_my_library:LED_D5.0mm
Changed lines of the file:
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@@
       (effects (font (size 1.27 1.27)) (justify right))
     )
-    (property "Footprint" "LED_THT:LED_D5.0mm" (at 114.3 55.88 0)
+    (property "Footprint" "01_my_library:LED_D5.0mm" (at 114.3 55.88 0)
       (effects (font (size 1.27 1.27)) hide)
     )
@@
       (effects (font (size 1.27 1.27)) (justify right))
     )
-    (property "Footprint" "LED_THT:LED_D5.0mm" (at 114.3 115.57 0)
+    (property "Footprint" "01_my_library:LED_D5.0mm" (at 114.3 115.57 0)
       (effects (font (size 1.27 1.27)) hide)
     )
@@
       (effects (font (size 1.27 1.27)) (justify right))
     )
-    (property "Footprint" "LED_THT:LED_D5.0mm" (at 237.49 125.73 0)
+    (property "Footprint" "01_my_library:LED_D5.0mm" (at 237.49 125.73 0)
       (effects (font (size 1.27 1.27)) hide)
     )
@@
       (effects (font (size 1.27 1.27)) (justify right))
     )
-    (property "Footprint" "LED_THT:LED_D5.0mm" (at 114.3 175.26 0)
-      (effects (font (size 1.27 1.27)) hide)
-    )
+    (property "Footprint" "01_my_library:LED_D5.0mm" (at 114.3 175.26 0)
+      (effects (font (size 1.27 1.27)) hide)
+    )
