File: control-logic.kicad_sch (KiCad schematic)
At the start: 3 parts, among them SW1 Button, U41 74HCT00

Commit message: kicad update
Parts:
- renumbered SW1 to SW7
Changed lines of the file:
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@@
   (symbol (lib_id "power:GND") (at 52.07 49.53 0) (unit 1)
     (in_bom yes) (on_board yes) (dnp no) (fields_autoplaced)
-    (property "Reference" "#PWR0175" (at 52.07 55.88 0)
+    (property "Reference" "#PWR0177" (at 52.07 55.88 0)
       (effects (font (size 1.27 1.27)) hide)
     )
@@
       (project "8-bit-cpu"
         (path "/100bb8d1-c3d6-4e1f-87b6-72e4e187243c/cbe1ebf3-0fd2-468b-b752-73c1c63eb76e"
-          (reference "#PWR0175") (unit 1)
+          (reference "#PWR0177") (unit 1)
         )
       )
@@
   (symbol (lib_id "Switch:SW_Push") (at 43.18 38.1 0) (unit 1)
     (in_bom yes) (on_board yes) (dnp no) (fields_autoplaced)
-    (property "Reference" "SW1" (at 43.18 30.48 0)
+    (property "Reference" "SW7" (at 43.18 30.48 0)
       (effects (font (size 1.27 1.27)))
     )
@@
     (instances
       (project "8-bit-cpu"
-        (path "/100bb8d1-c3d6-4e1f-87b6-72e4e187243c/45eb39c3-c748-461e-8330-08aae1247dee"
-          (reference "SW1") (unit 1)
-        )
-        (path "/100bb8d1-c3d6-4e1f-87b6-72e4e187243c/33b906b8-f63f-4a46-8ef2-4150917936b8/bcf72b05-a298-432c-8bad-dccda5c38b50"
-          (reference "SW6") (unit 1)
-        )
         (path "/100bb8d1-c3d6-4e1f-87b6-72e4e187243c/cbe1ebf3-0fd2-468b-b752-73c1c63eb76e"
           (reference "SW7") (unit 1)
@@
     (instances
       (project "8-bit-cpu"
-        (path "/100bb8d1-c3d6-4e1f-87b6-72e4e187243c/cbe1ebf3-0fd2-468b-b752-73c1c63eb76e/e9aea2e6-cf94-44c3-af7b-758fed303269"
-          (reference "U41") (unit 4)
-        )
         (path "/100bb8d1-c3d6-4e1f-87b6-72e4e187243c/cbe1ebf3-0fd2-468b-b752-73c1c63eb76e"
           (reference "U41") (unit 4)
@@
   (symbol (lib_id "power:+5V") (at 38.1 30.48 0) (unit 1)
     (in_bom yes) (on_board yes) (dnp no) (fields_autoplaced)
-    (property "Reference" "#PWR0174" (at 38.1 34.29 0)
+    (property "Reference" "#PWR0176" (at 38.1 34.29 0)
       (effects (font (size 1.27 1.27)) hide)
     )
@@
       (project "8-bit-cpu"
         (path "/100bb8d1-c3d6-4e1f-87b6-72e4e187243c/cbe1ebf3-0fd2-468b-b752-73c1c63eb76e"
-          (reference "#PWR0174") (unit 1)
+          (reference "#PWR0176") (unit 1)
         )
       )
@@
     (instances
       (project "8-bit-cpu"
-        (path "/100bb8d1-c3d6-4e1f-87b6-72e4e187243c/cbe1ebf3-0fd2-468b-b752-73c1c63eb76e/e9aea2e6-cf94-44c3-af7b-758fed303269"
-          (reference "U41") (unit 3)
-        )
         (path "/100bb8d1-c3d6-4e1f-87b6-72e4e187243c/cbe1ebf3-0fd2-468b-b752-73c1c63eb76e"
           (reference "U41") (unit 3)
