File: cpu-flags.kicad_sch (KiCad schematic)
At the start: 16 parts, among them U22 74HCT157, U50 74HCT02, U51 74HCT08, U53 74HCT08, U54 74HCT02, U9 74HCT173

Commit message: add arduino headers for programming
Parts:
- D106, D107: footprint (none) -> LED_THT:LED_D5.0mm
- R150, R151: footprint (none) -> Resistor_THT:R_Axial_DIN0204_L3.6mm_D1.6mm_P7.62mm_Horizontal
- U50, U51, U53, U54: footprint (none) -> Package_DIP:DIP-14_W7.62mm
Changed lines of the file:
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@@
       (effects (font (size 1.27 1.27)))
     )
-    (property "Footprint" "" (at 54.61 129.54 0)
+    (property "Footprint" "Package_DIP:DIP-14_W7.62mm" (at 54.61 129.54 0)
       (effects (font (size 1.27 1.27)) hide)
     )
@@
       (effects (font (size 1.27 1.27)) (justify left))
     )
-    (property "Footprint" "" (at 107.442 127 90)
+    (property "Footprint" "Resistor_THT:R_Axial_DIN0204_L3.6mm_D1.6mm_P7.62mm_Horizontal" (at 107.442 127 90)
       (effects (font (size 1.27 1.27)) hide)
     )
@@
       (effects (font (size 1.27 1.27)))
     )
-    (property "Footprint" "" (at 54.61 35.56 0)
+    (property "Footprint" "Package_DIP:DIP-14_W7.62mm" (at 54.61 35.56 0)
       (effects (font (size 1.27 1.27)) hide)
     )
@@
       (effects (font (size 1.27 1.27)))
     )
-    (property "Footprint" "" (at 54.61 144.78 0)
+    (property "Footprint" "Package_DIP:DIP-14_W7.62mm" (at 54.61 144.78 0)
       (effects (font (size 1.27 1.27)) hide)
     )
@@
       (effects (font (size 1.27 1.27)))
     )
-    (property "Footprint" "" (at 54.61 175.26 0)
+    (property "Footprint" "Package_DIP:DIP-14_W7.62mm" (at 54.61 175.26 0)
       (effects (font (size 1.27 1.27)) hide)
     )
@@
       (effects (font (size 1.27 1.27)) (justify left))
     )
-    (property "Footprint" "" (at 120.142 127 90)
+    (property "Footprint" "Resistor_THT:R_Axial_DIN0204_L3.6mm_D1.6mm_P7.62mm_Horizontal" (at 120.142 127 90)
       (effects (font (size 1.27 1.27)) hide)
     )
@@
       (effects (font (size 1.27 1.27)))
     )
-    (property "Footprint" "" (at 83.82 137.16 0)
+    (property "Footprint" "Package_DIP:DIP-14_W7.62mm" (at 83.82 137.16 0)
       (effects (font (size 1.27 1.27)) hide)
     )
@@
       (effects (font (size 1.27 1.27)))
     )
-    (property "Footprint" "" (at 113.03 152.4 0)
+    (property "Footprint" "Package_DIP:DIP-14_W7.62mm" (at 113.03 152.4 0)
       (effects (font (size 1.27 1.27)) hide)
     )
@@
       (effects (font (size 1.27 1.27)) (justify right))
     )
-    (property "Footprint" "" (at 121.92 119.38 0)
+    (property "Footprint" "LED_THT:LED_D5.0mm" (at 121.92 119.38 0)
       (effects (font (size 1.27 1.27)) hide)
     )
@@
       (effects (font (size 1.27 1.27)) (justify left))
     )
-    (property "Footprint" "" (at 265.43 82.55 0)
+    (property "Footprint" "Package_DIP:DIP-14_W7.62mm" (at 265.43 82.55 0)
       (effects (font (size 1.27 1.27)) hide)
     )
@@
       (effects (font (size 1.27 1.27)) (justify right))
     )
-    (property "Footprint" "" (at 109.22 119.38 0)
+    (property "Footprint" "LED_THT:LED_D5.0mm" (at 109.22 119.38 0)
       (effects (font (size 1.27 1.27)) hide)
     )
@@
       (effects (font (size 1.27 1.27)))
     )
-    (property "Footprint" "" (at 54.61 50.8 0)
+    (property "Footprint" "Package_DIP:DIP-14_W7.62mm" (at 54.61 50.8 0)
       (effects (font (size 1.27 1.27)) hide)
     )
@@
       (effects (font (size 1.27 1.27)))
     )
-    (property "Footprint" "" (at 237.49 124.46 0)
+    (property "Footprint" "Package_DIP:DIP-14_W7.62mm" (at 237.49 124.46 0)
       (effects (font (size 1.27 1.27)) hide)
     )
@@
       (effects (font (size 1.27 1.27)))
     )
-    (property "Footprint" "" (at 83.82 167.64 0)
+    (property "Footprint" "Package_DIP:DIP-14_W7.62mm" (at 83.82 167.64 0)
       (effects (font (size 1.27 1.27)) hide)
     )
@@
       (effects (font (size 1.27 1.27)))
     )
-    (property "Footprint" "" (at 83.82 73.66 0)
+    (property "Footprint" "Package_DIP:DIP-14_W7.62mm" (at 83.82 73.66 0)
       (effects (font (size 1.27 1.27)) hide)
     )
@@
       (effects (font (size 1.27 1.27)))
     )
-    (property "Footprint" "" (at 113.03 58.42 0)
+    (property "Footprint" "Package_DIP:DIP-14_W7.62mm" (at 113.03 58.42 0)
       (effects (font (size 1.27 1.27)) hide)
     )
@@
       (effects (font (size 1.27 1.27)))
     )
-    (property "Footprint" "" (at 260.35 124.46 0)
+    (property "Footprint" "Package_DIP:DIP-14_W7.62mm" (at 260.35 124.46 0)
       (effects (font (size 1.27 1.27)) hide)
     )
@@
       (effects (font (size 1.27 1.27)) (justify left))
     )
-    (property "Footprint" "" (at 237.49 41.91 0)
+    (property "Footprint" "Package_DIP:DIP-14_W7.62mm" (at 237.49 41.91 0)
       (effects (font (size 1.27 1.27)) hide)
     )
@@
       (effects (font (size 1.27 1.27)))
     )
-    (property "Footprint" "" (at 54.61 66.04 0)
+    (property "Footprint" "Package_DIP:DIP-14_W7.62mm" (at 54.61 66.04 0)
       (effects (font (size 1.27 1.27)) hide)
     )
@@
       (effects (font (size 1.27 1.27)) (justify left))
     )
-    (property "Footprint" "" (at 265.43 41.91 0)
+    (property "Footprint" "Package_DIP:DIP-14_W7.62mm" (at 265.43 41.91 0)
       (effects (font (size 1.27 1.27)) hide)
     )
@@
       (effects (font (size 1.27 1.27)) (justify left))
     )
-    (property "Footprint" "" (at 237.49 82.55 0)
+    (property "Footprint" "Package_DIP:DIP-14_W7.62mm" (at 237.49 82.55 0)
       (effects (font (size 1.27 1.27)) hide)
     )
@@
       (effects (font (size 1.27 1.27)))
     )
-    (property "Footprint" "" (at 54.61 160.02 0)
+    (property "Footprint" "Package_DIP:DIP-14_W7.62mm" (at 54.61 160.02 0)
       (effects (font (size 1.27 1.27)) hide)
     )
@@
       (effects (font (size 1.27 1.27)))
     )
-    (property "Footprint" "" (at 83.82 43.18 0)
+    (property "Footprint" "Package_DIP:DIP-14_W7.62mm" (at 83.82 43.18 0)
       (effects (font (size 1.27 1.27)) hide)
     )
@@
       (effects (font (size 1.27 1.27)))
     )
-    (property "Footprint" "" (at 54.61 81.28 0)
-      (effects (font (size 1.27 1.27)) hide)
-    )
+    (property "Footprint" "Package_DIP:DIP-14_W7.62mm" (at 54.61 81.28 0)
+      (effects (font (size 1.27 1.27)) hide)
+    )

Commit message: trying to solve issues
Parts:
- renumbered U50 to U52, U51 to U53, U53 to U55, U54 to U56
Connections:
- net ALU_ZERO: now also U22.14 (4A); no longer U22.13 (4B)
- net X_ZERO: now also U22.13 (4B); no longer U22.14 (4A)

Commit message: cleanup
Parts:
- renumbered D106 to D105, D107 to D106, R150 to R149, R151 to R150
Changed lines of the file:
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@@
         )
         (path "/100bb8d1-c3d6-4e1f-87b6-72e4e187243c/592ff0ed-0688-4db1-b04b-e905201025c7"
-          (reference "#PWR0222") (unit 1)
+          (reference "#PWR0221") (unit 1)
         )
       )
@@
         )
         (path "/100bb8d1-c3d6-4e1f-87b6-72e4e187243c/592ff0ed-0688-4db1-b04b-e905201025c7"
-          (reference "#PWR0232") (unit 1)
+          (reference "#PWR0231") (unit 1)
         )
       )
@@
   (symbol (lib_id "Device:R") (at 109.22 127 0) (unit 1)
     (in_bom yes) (on_board yes) (dnp no) (fields_autoplaced)
-    (property "Reference" "R150" (at 111.76 125.73 0)
+    (property "Reference" "R149" (at 111.76 125.73 0)
       (effects (font (size 1.27 1.27)) (justify left))
     )
@@
       (project "8-bit-cpu"
         (path "/100bb8d1-c3d6-4e1f-87b6-72e4e187243c/592ff0ed-0688-4db1-b04b-e905201025c7"
-          (reference "R150") (unit 1)
+          (reference "R149") (unit 1)
         )
       )
@@
         )
         (path "/100bb8d1-c3d6-4e1f-87b6-72e4e187243c/592ff0ed-0688-4db1-b04b-e905201025c7"
-          (reference "C62") (unit 1)
+          (reference "C61") (unit 1)
         )
       )
@@
         )
         (path "/100bb8d1-c3d6-4e1f-87b6-72e4e187243c/592ff0ed-0688-4db1-b04b-e905201025c7"
-          (reference "#PWR0214") (unit 1)
+          (reference "#PWR0213") (unit 1)
         )
       )
@@
   (symbol (lib_id "Device:R") (at 121.92 127 0) (unit 1)
     (in_bom yes) (on_board yes) (dnp no) (fields_autoplaced)
-    (property "Reference" "R151" (at 124.46 125.73 0)
+    (property "Reference" "R150" (at 124.46 125.73 0)
       (effects (font (size 1.27 1.27)) (justify left))
     )
@@
       (project "8-bit-cpu"
         (path "/100bb8d1-c3d6-4e1f-87b6-72e4e187243c/592ff0ed-0688-4db1-b04b-e905201025c7"
-          (reference "R151") (unit 1)
+          (reference "R150") (unit 1)
         )
       )
@@
         )
         (path "/100bb8d1-c3d6-4e1f-87b6-72e4e187243c/592ff0ed-0688-4db1-b04b-e905201025c7"
-          (reference "#PWR0223") (unit 1)
+          (reference "#PWR0222") (unit 1)
         )
       )
@@
         )
         (path "/100bb8d1-c3d6-4e1f-87b6-72e4e187243c/592ff0ed-0688-4db1-b04b-e905201025c7"
-          (reference "#PWR0217") (unit 1)
+          (reference "#PWR0216") (unit 1)
         )
       )
@@
         )
         (path "/100bb8d1-c3d6-4e1f-87b6-72e4e187243c/592ff0ed-0688-4db1-b04b-e905201025c7"
-          (reference "#PWR0228") (unit 1)
+          (reference "#PWR0227") (unit 1)
         )
       )
@@
         )
         (path "/100bb8d1-c3d6-4e1f-87b6-72e4e187243c/592ff0ed-0688-4db1-b04b-e905201025c7"
-          (reference "#PWR0230") (unit 1)
+          (reference "#PWR0229") (unit 1)
         )
       )
@@
         )
         (path "/100bb8d1-c3d6-4e1f-87b6-72e4e187243c/592ff0ed-0688-4db1-b04b-e905201025c7"
-          (reference "#PWR0231") (unit 1)
+          (reference "#PWR0230") (unit 1)
         )
       )
@@
         )
         (path "/100bb8d1-c3d6-4e1f-87b6-72e4e187243c/592ff0ed-0688-4db1-b04b-e905201025c7"
-          (reference "C63") (unit 1)
+          (reference "C62") (unit 1)
         )
       )
@@
         )
         (path "/100bb8d1-c3d6-4e1f-87b6-72e4e187243c/592ff0ed-0688-4db1-b04b-e905201025c7"
-          (reference "#PWR0215") (unit 1)
+          (reference "#PWR0214") (unit 1)
         )
       )
@@
   (symbol (lib_id "Device:LED") (at 121.92 119.38 90) (unit 1)
     (in_bom yes) (on_board yes) (dnp no) (fields_autoplaced)
-    (property "Reference" "D107" (at 125.73 119.6975 90)
+    (property "Reference" "D106" (at 125.73 119.6975 90)
       (effects (font (size 1.27 1.27)) (justify right))
     )
@@
       (project "8-bit-cpu"
         (path "/100bb8d1-c3d6-4e1f-87b6-72e4e187243c/592ff0ed-0688-4db1-b04b-e905201025c7"
-          (reference "D107") (unit 1)
+          (reference "D106") (unit 1)
         )
       )
@@
         )
         (path "/100bb8d1-c3d6-4e1f-87b6-72e4e187243c/592ff0ed-0688-4db1-b04b-e905201025c7"
-          (reference "#PWR0221") (unit 1)
+          (reference "#PWR0220") (unit 1)
         )
       )
@@
         )
         (path "/100bb8d1-c3d6-4e1f-87b6-72e4e187243c/592ff0ed-0688-4db1-b04b-e905201025c7"
-          (reference "#PWR0224") (unit 1)
+          (reference "#PWR0223") (unit 1)
         )
       )
@@
         )
         (path "/100bb8d1-c3d6-4e1f-87b6-72e4e187243c/592ff0ed-0688-4db1-b04b-e905201025c7"
-          (reference "#PWR0219") (unit 1)
+          (reference "#PWR0218") (unit 1)
         )
       )
@@
         )
         (path "/100bb8d1-c3d6-4e1f-87b6-72e4e187243c/592ff0ed-0688-4db1-b04b-e905201025c7"
-          (reference "C67") (unit 1)
+          (reference "C66") (unit 1)
         )
       )
@@
         )
         (path "/100bb8d1-c3d6-4e1f-87b6-72e4e187243c/592ff0ed-0688-4db1-b04b-e905201025c7"
-          (reference "C64") (unit 1)
+          (reference "C63") (unit 1)
         )
       )
@@
   (symbol (lib_id "Device:LED") (at 109.22 119.38 90) (unit 1)
     (in_bom yes) (on_board yes) (dnp no) (fields_autoplaced)
-    (property "Reference" "D106" (at 113.03 119.6975 90)
+    (property "Reference" "D105" (at 113.03 119.6975 90)
       (effects (font (size 1.27 1.27)) (justify right))
     )
@@
       (project "8-bit-cpu"
         (path "/100bb8d1-c3d6-4e1f-87b6-72e4e187243c/592ff0ed-0688-4db1-b04b-e905201025c7"
-          (reference "D106") (unit 1)
+          (reference "D105") (unit 1)
         )
       )
@@
         )
         (path "/100bb8d1-c3d6-4e1f-87b6-72e4e187243c/592ff0ed-0688-4db1-b04b-e905201025c7"
-          (reference "C65") (unit 1)
+          (reference "C64") (unit 1)
         )
       )
@@
         )
         (path "/100bb8d1-c3d6-4e1f-87b6-72e4e187243c/592ff0ed-0688-4db1-b04b-e905201025c7"
-          (reference "#PWR0220") (unit 1)
+          (reference "#PWR0219") (unit 1)
         )
       )
@@
   (symbol (lib_id "power:GND") (at 115.57 133.35 0) (unit 1)
     (in_bom yes) (on_board yes) (dnp no) (fields_autoplaced)
-    (property "Reference" "#PWR0234" (at 115.57 139.7 0)
+    (property "Reference" "#PWR0233" (at 115.57 139.7 0)
       (effects (font (size 1.27 1.27)) hide)
     )
@@
       (project "8-bit-cpu"
         (path "/100bb8d1-c3d6-4e1f-87b6-72e4e187243c/592ff0ed-0688-4db1-b04b-e905201025c7"
-          (reference "#PWR0234") (unit 1)
+          (reference "#PWR0233") (unit 1)
         )
       )
@@
         )
         (path "/100bb8d1-c3d6-4e1f-87b6-72e4e187243c/592ff0ed-0688-4db1-b04b-e905201025c7"
-          (reference "#PWR0216") (unit 1)
+          (reference "#PWR0215") (unit 1)
         )
       )
@@
         )
         (path "/100bb8d1-c3d6-4e1f-87b6-72e4e187243c/592ff0ed-0688-4db1-b04b-e905201025c7"
-          (reference "#PWR0229") (unit 1)
+          (reference "#PWR0228") (unit 1)
         )
       )
@@
         )
         (path "/100bb8d1-c3d6-4e1f-87b6-72e4e187243c/592ff0ed-0688-4db1-b04b-e905201025c7"
-          (reference "#PWR0218") (unit 1)
+          (reference "#PWR0217") (unit 1)
         )
       )
@@
         )
         (path "/100bb8d1-c3d6-4e1f-87b6-72e4e187243c/592ff0ed-0688-4db1-b04b-e905201025c7"
-          (reference "#PWR0225") (unit 1)
+          (reference "#PWR0224") (unit 1)
         )
       )
@@
         )
         (path "/100bb8d1-c3d6-4e1f-87b6-72e4e187243c/592ff0ed-0688-4db1-b04b-e905201025c7"
-          (reference "#PWR0227") (unit 1)
+          (reference "#PWR0226") (unit 1)
         )
       )
@@
         )
         (path "/100bb8d1-c3d6-4e1f-87b6-72e4e187243c/592ff0ed-0688-4db1-b04b-e905201025c7"
-          (reference "#PWR0226") (unit 1)
+          (reference "#PWR0225") (unit 1)
         )
       )
@@
         )
         (path "/100bb8d1-c3d6-4e1f-87b6-72e4e187243c/592ff0ed-0688-4db1-b04b-e905201025c7"
-          (reference "#PWR0233") (unit 1)
+          (reference "#PWR0232") (unit 1)
         )
       )
@@
         )
         (path "/100bb8d1-c3d6-4e1f-87b6-72e4e187243c/592ff0ed-0688-4db1-b04b-e905201025c7"
-          (reference "C66") (unit 1)
-        )
-      )
+          (reference "C65") (unit 1)
+        )
+      )

Commit message: readme
Parts:
- added C13: 10n, 01_my_library:C_Disc_D4.0mm_W2.6mm_P2.50mm, symbol Device:C
Connections:
- net GND: now also C13.2
- net RESET: now also C13.1
Changed lines of the file:
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@@
   (junction (at 151.13 53.34) (diameter 0) (color 0 0 0 0)
+  )
+  (junction (at 127 71.12) (diameter 0) (color 255 0 0 1)
   )
   (junction (at 109.22 111.76) (diameter 0) (color 0 0 0 0)
@@
     (stroke (width 0) (type default))
   )
+  (wire (pts (xy 127 60.96) (xy 133.35 60.96))
+    (stroke (width 0) (type default) (color 255 0 0 1))
+  )
   (wire (pts (xy 229.87 121.92) (xy 229.87 127))
     (stroke (width 0) (type default))
@@
     (stroke (width 0) (type default))
   )
+  (wire (pts (xy 133.35 60.96) (xy 133.35 62.23))
+    (stroke (width 0) (type default) (color 255 0 0 1))
+  )
   (wire (pts (xy 142.24 81.28) (xy 144.78 81.28))
     (stroke (width 0) (type default))
@@
   (wire (pts (xy 191.77 38.1) (xy 189.23 38.1))
     (stroke (width 0) (type default))
+  )
+  (wire (pts (xy 127 71.12) (xy 127 60.96))
+    (stroke (width 0) (type default) (color 255 0 0 1))
   )
   (wire (pts (xy 33.02 67.31) (xy 38.1 67.31))
@@
   (hierarchical_label "X_2" (shape input) (at 33.02 148.59 180) (fields_autoplaced)
     (effects (font (size 1.27 1.27)) (justify right))
+  )
+  (symbol (lib_id "Device:C") (at 133.35 66.04 0) (unit 1)
+    (in_bom yes) (on_board yes) (dnp yes) (fields_autoplaced)
+    (property "Reference" "C13" (at 137.16 64.77 0)
+      (effects (font (size 1.27 1.27)) (justify left))
+    )
+    (property "Value" "10n" (at 137.16 67.31 0)
+      (effects (font (size 1.27 1.27)) (justify left))
+    )
+    (property "Footprint" "01_my_library:C_Disc_D4.0mm_W2.6mm_P2.50mm" (at 134.3152 69.85 0)
+      (effects (font (size 1.27 1.27)) hide)
+    )
+    (property "Datasheet" "~" (at 133.35 66.04 0)
+      (effects (font (size 1.27 1.27)) hide)
+    )
+    (pin "1")
+    (pin "2")
+    (instances
+      (project "8-bit-cpu"
+        (path "/100bb8d1-c3d6-4e1f-87b6-72e4e187243c/651dfbaf-e340-4976-8216-793c5a5aaa3b"
+          (reference "C13") (unit 1)
+        )
+        (path "/100bb8d1-c3d6-4e1f-87b6-72e4e187243c/592ff0ed-0688-4db1-b04b-e905201025c7"
+          (reference "C81") (unit 1)
+        )
+      )
+    )
   )
   (symbol (lib_id "74xx:74HCT02") (at 54.61 129.54 0) (unit 1)
@@
         )
       )
+    )
+  )
+  (symbol (lib_id "power:GND") (at 133.35 69.85 0) (unit 1)
+    (in_bom yes) (on_board yes) (dnp no) (fields_autoplaced)
+    (property "Reference" "#PWR03" (at 133.35 76.2 0)
+      (effects (font (size 1.27 1.27)) hide)
+    )
+    (property "Value" "GND" (at 133.35 74.93 0)
+      (effects (font (size 1.27 1.27)) hide)
+    )
+    (property "Footprint" "" (at 133.35 69.85 0)
+      (effects (font (size 1.27 1.27)) hide)
+    )
+    (property "Datasheet" "" (at 133.35 69.85 0)
+      (effects (font (size 1.27 1.27)) hide)
+    )
+    (pin "1")
+    (instances
+      (project "8-bit-cpu"
+        (path "/100bb8d1-c3d6-4e1f-87b6-72e4e187243c/45eb39c3-c748-461e-8330-08aae1247dee"
+          (reference "#PWR03") (unit 1)
+        )
+        (path "/100bb8d1-c3d6-4e1f-87b6-72e4e187243c/651dfbaf-e340-4976-8216-793c5a5aaa3b"
+          (reference "#PWR038") (unit 1)
+        )
+        (path "/100bb8d1-c3d6-4e1f-87b6-72e4e187243c/3568514a-e420-48fa-9fd5-7a290120765b"
+          (reference "#PWR056") (unit 1)
+        )
+        (path "/100bb8d1-c3d6-4e1f-87b6-72e4e187243c/592ff0ed-0688-4db1-b04b-e905201025c7"
+          (reference "#PWR0269") (unit 1)
+        )
+      )
