File: eeprom-address-buffer.kicad_sch (KiCad schematic)
At the start: 4 parts, among them U8 74HCT173

Commit message: readme
Parts:
- added C13: 10n, 01_my_library:C_Disc_D4.0mm_W2.6mm_P2.50mm, symbol Device:C
Connections:
- net GND: now also C13.2
- net RESET: now also C13.1
Changed lines of the file:
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@@
   (junction (at 111.76 80.01) (diameter 0) (color 0 0 0 0)
   )
+  (junction (at 182.88 76.2) (diameter 0) (color 255 0 0 1)
+  )
   (junction (at 148.59 95.25) (diameter 0) (color 0 0 0 0)
   )
@@
     (stroke (width 0) (type default))
   )
+  (wire (pts (xy 182.88 62.23) (xy 195.58 62.23))
+    (stroke (width 0) (type default) (color 255 0 0 1))
+  )
   (wire (pts (xy 82.55 69.85) (xy 124.46 69.85))
     (stroke (width 0) (type default))
@@
     (stroke (width 0) (type default))
   )
+  (wire (pts (xy 182.88 76.2) (xy 182.88 62.23))
+    (stroke (width 0) (type default) (color 255 0 0 1))
+  )
   (wire (pts (xy 190.5 80.01) (xy 190.5 82.55))
     (stroke (width 0) (type default))
@@
   (wire (pts (xy 82.55 67.31) (xy 127 67.31))
     (stroke (width 0) (type default))
+  )
+  (wire (pts (xy 195.58 62.23) (xy 195.58 64.77))
+    (stroke (width 0) (type default) (color 255 0 0 1))
   )
   (wire (pts (xy 132.08 62.23) (xy 132.08 82.55))
@@
     )
   )
+  (symbol (lib_id "power:GND") (at 195.58 72.39 0) (unit 1)
+    (in_bom yes) (on_board yes) (dnp no) (fields_autoplaced)
+    (property "Reference" "#PWR03" (at 195.58 78.74 0)
+      (effects (font (size 1.27 1.27)) hide)
+    )
+    (property "Value" "GND" (at 195.58 77.47 0)
+      (effects (font (size 1.27 1.27)) hide)
+    )
+    (property "Footprint" "" (at 195.58 72.39 0)
+      (effects (font (size 1.27 1.27)) hide)
+    )
+    (property "Datasheet" "" (at 195.58 72.39 0)
+      (effects (font (size 1.27 1.27)) hide)
+    )
+    (pin "1")
+    (instances
+      (project "8-bit-cpu"
+        (path "/100bb8d1-c3d6-4e1f-87b6-72e4e187243c/45eb39c3-c748-461e-8330-08aae1247dee"
+          (reference "#PWR03") (unit 1)
+        )
+        (path "/100bb8d1-c3d6-4e1f-87b6-72e4e187243c/651dfbaf-e340-4976-8216-793c5a5aaa3b"
+          (reference "#PWR038") (unit 1)
+        )
+        (path "/100bb8d1-c3d6-4e1f-87b6-72e4e187243c/3568514a-e420-48fa-9fd5-7a290120765b"
+          (reference "#PWR056") (unit 1)
+        )
+        (path "/100bb8d1-c3d6-4e1f-87b6-72e4e187243c/cbe1ebf3-0fd2-468b-b752-73c1c63eb76e/da230027-cd37-47f3-abaf-a6951a86af11"
+          (reference "#PWR0268") (unit 1)
+        )
+      )
+    )
+  )
   (symbol (lib_id "power:+5V") (at 148.59 92.71 0) (unit 1)
     (in_bom yes) (on_board yes) (dnp no) (fields_autoplaced)
@@
         )
       )
+    )
+  )
+  (symbol (lib_id "Device:C") (at 195.58 68.58 0) (unit 1)
+    (in_bom yes) (on_board yes) (dnp yes) (fields_autoplaced)
+    (property "Reference" "C13" (at 199.39 67.31 0)
+      (effects (font (size 1.27 1.27)) (justify left))
+    )
+    (property "Value" "10n" (at 199.39 69.85 0)
+      (effects (font (size 1.27 1.27)) (justify left))
+    )
+    (property "Footprint" "01_my_library:C_Disc_D4.0mm_W2.6mm_P2.50mm" (at 196.5452 72.39 0)
+      (effects (font (size 1.27 1.27)) hide)
+    )
+    (property "Datasheet" "~" (at 195.58 68.58 0)
+      (effects (font (size 1.27 1.27)) hide)
+    )
+    (pin "1")
+    (pin "2")
+    (instances
+      (project "8-bit-cpu"
+        (path "/100bb8d1-c3d6-4e1f-87b6-72e4e187243c/651dfbaf-e340-4976-8216-793c5a5aaa3b"
+          (reference "C13") (unit 1)
+        )
+        (path "/100bb8d1-c3d6-4e1f-87b6-72e4e187243c/cbe1ebf3-0fd2-468b-b752-73c1c63eb76e/da230027-cd37-47f3-abaf-a6951a86af11"
+          (reference "C80") (unit 1)
+        )
+      )

Commit message: kicad update
Parts:
- renumbered C13 to C54, C1 to C55, C1 to C56, U8 to U42, U8 to U43
