File: instruction-register.kicad_sch (KiCad schematic)
At the start: 20 parts, among them U8 74HCT173, U9 74HCT173

Commit message: readme
Parts:
- added C13: 10n, 01_my_library:C_Disc_D4.0mm_W2.6mm_P2.50mm, symbol Device:C
Connections:
- net GND: now also C13.2
- net RESET: now also C13.1
Changed lines of the file:
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@@
   (junction (at 107.95 71.12) (diameter 0) (color 255 0 0 1)
   )
+  (junction (at 161.29 58.42) (diameter 0) (color 255 0 0 1)
+  )
   (junction (at 120.65 160.02) (diameter 0) (color 0 0 0 0)
   )
@@
     (stroke (width 0) (type default) (color 0 0 255 1))
   )
+  (wire (pts (xy 161.29 58.42) (xy 161.29 46.99))
+    (stroke (width 0) (type default) (color 255 0 0 1))
+  )
   (wire (pts (xy 208.28 82.55) (xy 208.28 81.28))
     (stroke (width 0) (type default))
@@
     (stroke (width 0) (type default) (color 255 0 0 1))
   )
+  (wire (pts (xy 161.29 46.99) (xy 175.26 46.99))
+    (stroke (width 0) (type default) (color 255 0 0 1))
+  )
   (wire (pts (xy 184.15 97.79) (xy 184.15 110.49))
     (stroke (width 0) (type default))
@@
   (wire (pts (xy 58.42 44.45) (xy 184.15 44.45))
     (stroke (width 0) (type default) (color 0 0 255 1))
+  )
+  (wire (pts (xy 175.26 46.99) (xy 175.26 49.53))
+    (stroke (width 0) (type default) (color 255 0 0 1))
   )
   (wire (pts (xy 135.89 81.28) (xy 135.89 85.09))
@@
     )
   )
+  (symbol (lib_id "power:GND") (at 175.26 57.15 0) (unit 1)
+    (in_bom yes) (on_board yes) (dnp no) (fields_autoplaced)
+    (property "Reference" "#PWR03" (at 175.26 63.5 0)
+      (effects (font (size 1.27 1.27)) hide)
+    )
+    (property "Value" "GND" (at 175.26 62.23 0)
+      (effects (font (size 1.27 1.27)) hide)
+    )
+    (property "Footprint" "" (at 175.26 57.15 0)
+      (effects (font (size 1.27 1.27)) hide)
+    )
+    (property "Datasheet" "" (at 175.26 57.15 0)
+      (effects (font (size 1.27 1.27)) hide)
+    )
+    (pin "1")
+    (instances
+      (project "8-bit-cpu"
+        (path "/100bb8d1-c3d6-4e1f-87b6-72e4e187243c/45eb39c3-c748-461e-8330-08aae1247dee"
+          (reference "#PWR03") (unit 1)
+        )
+        (path "/100bb8d1-c3d6-4e1f-87b6-72e4e187243c/651dfbaf-e340-4976-8216-793c5a5aaa3b"
+          (reference "#PWR038") (unit 1)
+        )
+        (path "/100bb8d1-c3d6-4e1f-87b6-72e4e187243c/3568514a-e420-48fa-9fd5-7a290120765b"
+          (reference "#PWR056") (unit 1)
+        )
+        (path "/100bb8d1-c3d6-4e1f-87b6-72e4e187243c/1f5609ed-b95d-46c8-9fbb-4fdf6df08011"
+          (reference "#PWR0267") (unit 1)
+        )
+      )
+    )
+  )
   (symbol (lib_id "power:GND") (at 90.17 85.09 0) (unit 1)
     (in_bom yes) (on_board yes) (dnp no) (fields_autoplaced)
@@
         )
       )
+    )
+  )
+  (symbol (lib_id "Device:C") (at 175.26 53.34 0) (unit 1)
+    (in_bom yes) (on_board yes) (dnp yes) (fields_autoplaced)
+    (property "Reference" "C13" (at 179.07 52.07 0)
+      (effects (font (size 1.27 1.27)) (justify left))
+    )
+    (property "Value" "10n" (at 179.07 54.61 0)
+      (effects (font (size 1.27 1.27)) (justify left))
+    )
+    (property "Footprint" "01_my_library:C_Disc_D4.0mm_W2.6mm_P2.50mm" (at 176.2252 57.15 0)
+      (effects (font (size 1.27 1.27)) hide)
+    )
+    (property "Datasheet" "~" (at 175.26 53.34 0)
+      (effects (font (size 1.27 1.27)) hide)
+    )
+    (pin "1")
+    (pin "2")
+    (instances
+      (project "8-bit-cpu"
+        (path "/100bb8d1-c3d6-4e1f-87b6-72e4e187243c/651dfbaf-e340-4976-8216-793c5a5aaa3b"
+          (reference "C13") (unit 1)
+        )
+        (path "/100bb8d1-c3d6-4e1f-87b6-72e4e187243c/1f5609ed-b95d-46c8-9fbb-4fdf6df08011"
+          (reference "C79") (unit 1)
+        )
+      )

Commit message: kicad update
Parts:
- D64: renamed from D5; footprint LED_THT:LED_D5.0mm -> 01_my_library:LED_D5.0mm
- D65: renamed from D6; footprint LED_THT:LED_D5.0mm -> 01_my_library:LED_D5.0mm
- D66: renamed from D7; footprint LED_THT:LED_D5.0mm -> 01_my_library:LED_D5.0mm
- D67: renamed from D8; footprint LED_THT:LED_D5.0mm -> 01_my_library:LED_D5.0mm
- D68: renamed from D9; footprint LED_THT:LED_D5.0mm -> 01_my_library:LED_D5.0mm
- D69: renamed from D10; footprint LED_THT:LED_D5.0mm -> 01_my_library:LED_D5.0mm
- D70: renamed from D11; footprint LED_THT:LED_D5.0mm -> 01_my_library:LED_D5.0mm
- D71: renamed from D12; footprint LED_THT:LED_D5.0mm -> 01_my_library:LED_D5.0mm
- renumbered C13 to C51, C1 to C52, C1 to C53, R11 to R107, R12 to R108, R13 to R109, R14 to R110, R15 to R111, R16 to R112, R17 to R113, R18 to R114, U9 to U39, U8 to U40
