File: left-microcode-eeprom.kicad_sch (KiCad schematic)
At the start: 20 parts, among them U37 AT28C64B, U49 74HCT04

Commit message: add pdf for instructions
Other:
- company: (none) -> TBR Designs
- title: (none) -> 8-bit CPU
Changed lines of the file:
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@@
 (kicad_sch (version 20230121) (generator eeschema)
   (paper "A4")
+  (title_block
+    (title "8-bit CPU")
+    (date "2023-11-28")
+    (rev "1.0")
+    (company "TBR Designs")
+  )
   (junction (at 158.75 111.76) (diameter 0) (color 0 0 0 0)
   )

Commit message: some cleanup
Parts:
- renumbered U49 to U44

Commit message: add arduino headers for programming
Parts:
- U44: footprint (none) -> Package_DIP:DIP-14_W7.62mm
Changed lines of the file:
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@@
       (effects (font (size 1.27 1.27)))
     )
-    (property "Footprint" "" (at 73.66 106.68 0)
+    (property "Footprint" "Package_DIP:DIP-14_W7.62mm" (at 73.66 106.68 0)
       (effects (font (size 1.27 1.27)) hide)
     )
@@
       (effects (font (size 1.27 1.27)))
     )
-    (property "Footprint" "" (at 73.66 120.65 0)
+    (property "Footprint" "Package_DIP:DIP-14_W7.62mm" (at 73.66 120.65 0)
       (effects (font (size 1.27 1.27)) hide)
     )
@@
       (effects (font (size 1.27 1.27)))
     )
-    (property "Footprint" "" (at 73.66 148.59 0)
+    (property "Footprint" "Package_DIP:DIP-14_W7.62mm" (at 73.66 148.59 0)
       (effects (font (size 1.27 1.27)) hide)
     )
@@
       (effects (font (size 1.27 1.27)))
     )
-    (property "Footprint" "" (at 73.66 162.56 0)
+    (property "Footprint" "Package_DIP:DIP-14_W7.62mm" (at 73.66 162.56 0)
       (effects (font (size 1.27 1.27)) hide)
     )
@@
       (effects (font (size 1.27 1.27)) (justify left))
     )
-    (property "Footprint" "" (at 257.81 38.1 0)
+    (property "Footprint" "Package_DIP:DIP-14_W7.62mm" (at 257.81 38.1 0)
       (effects (font (size 1.27 1.27)) hide)
     )
@@
       (effects (font (size 1.27 1.27)))
     )
-    (property "Footprint" "" (at 73.66 134.62 0)
+    (property "Footprint" "Package_DIP:DIP-14_W7.62mm" (at 73.66 134.62 0)
       (effects (font (size 1.27 1.27)) hide)
     )
@@
       (effects (font (size 1.27 1.27)))
     )
-    (property "Footprint" "" (at 73.66 92.71 0)
-      (effects (font (size 1.27 1.27)) hide)
-    )
+    (property "Footprint" "Package_DIP:DIP-14_W7.62mm" (at 73.66 92.71 0)
+      (effects (font (size 1.27 1.27)) hide)
+    )

Commit message: cleanup
Parts:
- D10, D11, D12, D5, D6, D7, D8, D9: value YELLOW -> BLUE
Changed lines of the file:
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@@
         )
         (path "/100bb8d1-c3d6-4e1f-87b6-72e4e187243c/cbe1ebf3-0fd2-468b-b752-73c1c63eb76e/0e5af4fe-5ef2-4486-974c-49740f34623a"
-          (reference "#PWR0184") (unit 1)
+          (reference "#PWR0187") (unit 1)
         )
       )
@@
       (effects (font (size 1.27 1.27)) (justify right))
     )
-    (property "Value" "YELLOW" (at 203.2 135.89 90)
+    (property "Value" "BLUE" (at 203.2 135.89 90)
       (effects (font (size 1.27 1.27)) (justify right))
     )
@@
         )
         (path "/100bb8d1-c3d6-4e1f-87b6-72e4e187243c/cbe1ebf3-0fd2-468b-b752-73c1c63eb76e/0e5af4fe-5ef2-4486-974c-49740f34623a"
-          (reference "#PWR0182") (unit 1)
+          (reference "#PWR0185") (unit 1)
         )
       )
@@
       (effects (font (size 1.27 1.27)) (justify right))
     )
-    (property "Value" "YELLOW" (at 243.84 135.89 90)
+    (property "Value" "BLUE" (at 243.84 135.89 90)
       (effects (font (size 1.27 1.27)) (justify right))
     )
@@
         )
         (path "/100bb8d1-c3d6-4e1f-87b6-72e4e187243c/cbe1ebf3-0fd2-468b-b752-73c1c63eb76e/0e5af4fe-5ef2-4486-974c-49740f34623a"
-          (reference "#PWR0188") (unit 1)
+          (reference "#PWR0191") (unit 1)
         )
       )
@@
         )
         (path "/100bb8d1-c3d6-4e1f-87b6-72e4e187243c/cbe1ebf3-0fd2-468b-b752-73c1c63eb76e/0e5af4fe-5ef2-4486-974c-49740f34623a"
-          (reference "#PWR0186") (unit 1)
+          (reference "#PWR0189") (unit 1)
         )
       )
@@
         )
         (path "/100bb8d1-c3d6-4e1f-87b6-72e4e187243c/cbe1ebf3-0fd2-468b-b752-73c1c63eb76e/0e5af4fe-5ef2-4486-974c-49740f34623a"
-          (reference "#PWR0185") (unit 1)
+          (reference "#PWR0188") (unit 1)
         )
       )
@@
       (effects (font (size 1.27 1.27)) (justify right))
     )
-    (property "Value" "YELLOW" (at 223.52 135.89 90)
+    (property "Value" "BLUE" (at 223.52 135.89 90)
       (effects (font (size 1.27 1.27)) (justify right))
     )
@@
       (effects (font (size 1.27 1.27)) (justify right))
     )
-    (property "Value" "YELLOW" (at 193.04 135.89 90)
+    (property "Value" "BLUE" (at 193.04 135.89 90)
       (effects (font (size 1.27 1.27)) (justify right))
     )
@@
         )
         (path "/100bb8d1-c3d6-4e1f-87b6-72e4e187243c/cbe1ebf3-0fd2-468b-b752-73c1c63eb76e/0e5af4fe-5ef2-4486-974c-49740f34623a"
-          (reference "#PWR0187") (unit 1)
+          (reference "#PWR0190") (unit 1)
         )
       )
@@
       (effects (font (size 1.27 1.27)) (justify right))
     )
-    (property "Value" "YELLOW" (at 264.16 135.89 90)
+    (property "Value" "BLUE" (at 264.16 135.89 90)
       (effects (font (size 1.27 1.27)) (justify right))
     )
@@
         )
         (path "/100bb8d1-c3d6-4e1f-87b6-72e4e187243c/cbe1ebf3-0fd2-468b-b752-73c1c63eb76e/0e5af4fe-5ef2-4486-974c-49740f34623a"
-          (reference "#PWR0183") (unit 1)
+          (reference "#PWR0186") (unit 1)
         )
       )
@@
       (effects (font (size 1.27 1.27)) (justify right))
     )
-    (property "Value" "YELLOW" (at 233.68 135.89 90)
+    (property "Value" "BLUE" (at 233.68 135.89 90)
       (effects (font (size 1.27 1.27)) (justify right))
     )
@@
       (effects (font (size 1.27 1.27)) (justify right))
     )
-    (property "Value" "YELLOW" (at 254 135.89 90)
+    (property "Value" "BLUE" (at 254 135.89 90)
       (effects (font (size 1.27 1.27)) (justify right))
     )
@@
       (effects (font (size 1.27 1.27)) (justify right))
     )
-    (property "Value" "YELLOW" (at 213.36 135.89 90)
-      (effects (font (size 1.27 1.27)) (justify right))
-    )
+    (property "Value" "BLUE" (at 213.36 135.89 90)
+      (effects (font (size 1.27 1.27)) (justify right))
+    )

Commit message: trying to solve issues
Parts:
- renumbered U44 to U46
Connections:
- net CARRY_FLAG renamed EEPROM_9
- net INSTRUCTION_0 renamed EEPROM_3
- net INSTRUCTION_1 renamed EEPROM_4
- net INSTRUCTION_2 renamed EEPROM_5
- net INSTRUCTION_3 renamed EEPROM_6
- net INSTRUCTION_4 renamed EEPROM_7
- net INSTRUCTION_5 renamed EEPROM_8
- net ZERO_FLAG renamed EEPROM_10
Changed lines of the file:
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@@
     (effects (font (size 1.27 1.27)) (justify left bottom))
   )
+  (hierarchical_label "EEPROM_8" (shape input) (at 41.91 38.1 180) (fields_autoplaced)
+    (effects (font (size 1.27 1.27)) (justify right))
+  )
   (hierarchical_label "RAM_INPUT" (shape output) (at 41.91 81.28 180) (fields_autoplaced)
     (effects (font (size 1.27 1.27)) (justify right))
   )
-  (hierarchical_label "INSTRUCTION_0" (shape input) (at 41.91 25.4 180) (fields_autoplaced)
+  (hierarchical_label "EEPROM_3" (shape input) (at 41.91 25.4 180) (fields_autoplaced)
     (effects (font (size 1.27 1.27)) (justify right))
   )
@@
     (effects (font (size 1.27 1.27)) (justify right))
   )
-  (hierarchical_label "INSTRUCTION_1" (shape input) (at 41.91 27.94 180) (fields_autoplaced)
-    (effects (font (size 1.27 1.27)) (justify right))
-  )
-  (hierarchical_label "INSTRUCTION_3" (shape input) (at 41.91 33.02 180) (fields_autoplaced)
-    (effects (font (size 1.27 1.27)) (justify right))
-  )
-  (hierarchical_label "ZERO_FLAG" (shape input) (at 41.91 43.18 180) (fields_autoplaced)
+  (hierarchical_label "EEPROM_9" (shape input) (at 41.91 40.64 180) (fields_autoplaced)
     (effects (font (size 1.27 1.27)) (justify right))
   )
@@
     (effects (font (size 1.27 1.27)) (justify right))
   )
-  (hierarchical_label "INSTRUCTION_5" (shape input) (at 41.91 38.1 180) (fields_autoplaced)
+  (hierarchical_label "EEPROM_4" (shape input) (at 41.91 27.94 180) (fields_autoplaced)
     (effects (font (size 1.27 1.27)) (justify right))
   )
@@
     (effects (font (size 1.27 1.27)) (justify right))
   )
-  (hierarchical_label "INSTRUCTION_4" (shape input) (at 41.91 35.56 180) (fields_autoplaced)
-    (effects (font (size 1.27 1.27)) (justify right))
-  )
-  (hierarchical_label "CARRY_FLAG" (shape input) (at 41.91 40.64 180) (fields_autoplaced)
-    (effects (font (size 1.27 1.27)) (justify right))
-  )
-  (hierarchical_label "INSTRUCTION_2" (shape input) (at 41.91 30.48 180) (fields_autoplaced)
+  (hierarchical_label "EEPROM_6" (shape input) (at 41.91 33.02 180) (fields_autoplaced)
     (effects (font (size 1.27 1.27)) (justify right))
   )
   (hierarchical_label "COUNT_ENABLE" (shape output) (at 41.91 78.74 180) (fields_autoplaced)
+    (effects (font (size 1.27 1.27)) (justify right))
+  )
+  (hierarchical_label "EEPROM_7" (shape input) (at 41.91 35.56 180) (fields_autoplaced)
+    (effects (font (size 1.27 1.27)) (justify right))
+  )
+  (hierarchical_label "EEPROM_5" (shape input) (at 41.91 30.48 180) (fields_autoplaced)
+    (effects (font (size 1.27 1.27)) (justify right))
+  )
+  (hierarchical_label "EEPROM_10" (shape input) (at 41.91 43.18 180) (fields_autoplaced)
     (effects (font (size 1.27 1.27)) (justify right))
   )
@@
         )
         (path "/100bb8d1-c3d6-4e1f-87b6-72e4e187243c/cbe1ebf3-0fd2-468b-b752-73c1c63eb76e/0e5af4fe-5ef2-4486-974c-49740f34623a"
-          (reference "U45") (unit 1)
+          (reference "U47") (unit 1)
         )
       )
@@
   (symbol (lib_id "74xx:74HCT04") (at 73.66 106.68 180) (unit 2)
     (in_bom yes) (on_board yes) (dnp no) (fields_autoplaced)
-    (property "Reference" "U44" (at 73.66 97.79 0)
+    (property "Reference" "U46" (at 73.66 97.79 0)
       (effects (font (size 1.27 1.27)))
     )
@@
       (project "8-bit-cpu"
         (path "/100bb8d1-c3d6-4e1f-87b6-72e4e187243c/cbe1ebf3-0fd2-468b-b752-73c1c63eb76e/0e5af4fe-5ef2-4486-974c-49740f34623a"
-          (reference "U44") (unit 2)
+          (reference "U46") (unit 2)
         )
       )
@@
         )
         (path "/100bb8d1-c3d6-4e1f-87b6-72e4e187243c/cbe1ebf3-0fd2-468b-b752-73c1c63eb76e/0e5af4fe-5ef2-4486-974c-49740f34623a"
-          (reference "#PWR0187") (unit 1)
+          (reference "#PWR0194") (unit 1)
         )
       )
@@
         )
         (path "/100bb8d1-c3d6-4e1f-87b6-72e4e187243c/cbe1ebf3-0fd2-468b-b752-73c1c63eb76e/0e5af4fe-5ef2-4486-974c-49740f34623a"
-          (reference "C52") (unit 1)
+          (reference "C56") (unit 1)
         )
       )
@@
   (symbol (lib_id "74xx:74HCT04") (at 73.66 120.65 180) (unit 3)
     (in_bom yes) (on_board yes) (dnp no) (fields_autoplaced)
-    (property "Reference" "U44" (at 73.66 111.76 0)
+    (property "Reference" "U46" (at 73.66 111.76 0)
       (effects (font (size 1.27 1.27)))
     )
@@
       (project "8-bit-cpu"
         (path "/100bb8d1-c3d6-4e1f-87b6-72e4e187243c/cbe1ebf3-0fd2-468b-b752-73c1c63eb76e/0e5af4fe-5ef2-4486-974c-49740f34623a"
-          (reference "U44") (unit 3)
+          (reference "U46") (unit 3)
         )
       )
@@
         )
         (path "/100bb8d1-c3d6-4e1f-87b6-72e4e187243c/cbe1ebf3-0fd2-468b-b752-73c1c63eb76e/0e5af4fe-5ef2-4486-974c-49740f34623a"
-          (reference "#PWR0185") (unit 1)
+          (reference "#PWR0192") (unit 1)
         )
       )
@@
   (symbol (lib_id "74xx:74HCT04") (at 73.66 148.59 180) (unit 5)
     (in_bom yes) (on_board yes) (dnp no) (fields_autoplaced)
-    (property "Reference" "U44" (at 73.66 139.7 0)
+    (property "Reference" "U46" (at 73.66 139.7 0)
       (effects (font (size 1.27 1.27)))
     )
@@
       (project "8-bit-cpu"
         (path "/100bb8d1-c3d6-4e1f-87b6-72e4e187243c/cbe1ebf3-0fd2-468b-b752-73c1c63eb76e/0e5af4fe-5ef2-4486-974c-49740f34623a"
-          (reference "U44") (unit 5)
+          (reference "U46") (unit 5)
         )
       )
@@
   (symbol (lib_id "74xx:74HCT04") (at 73.66 162.56 180) (unit 6)
     (in_bom yes) (on_board yes) (dnp no) (fields_autoplaced)
-    (property "Reference" "U44" (at 73.66 153.67 0)
+    (property "Reference" "U46" (at 73.66 153.67 0)
       (effects (font (size 1.27 1.27)))
     )
@@
       (project "8-bit-cpu"
         (path "/100bb8d1-c3d6-4e1f-87b6-72e4e187243c/cbe1ebf3-0fd2-468b-b752-73c1c63eb76e/0e5af4fe-5ef2-4486-974c-49740f34623a"
-          (reference "U44") (unit 6)
+          (reference "U46") (unit 6)
         )
       )
@@
         )
         (path "/100bb8d1-c3d6-4e1f-87b6-72e4e187243c/cbe1ebf3-0fd2-468b-b752-73c1c63eb76e/0e5af4fe-5ef2-4486-974c-49740f34623a"
-          (reference "#PWR0191") (unit 1)
+          (reference "#PWR0198") (unit 1)
         )
       )
@@
         )
         (path "/100bb8d1-c3d6-4e1f-87b6-72e4e187243c/cbe1ebf3-0fd2-468b-b752-73c1c63eb76e/0e5af4fe-5ef2-4486-974c-49740f34623a"
-          (reference "#PWR0189") (unit 1)
+          (reference "#PWR0196") (unit 1)
         )
       )
@@
         )
         (path "/100bb8d1-c3d6-4e1f-87b6-72e4e187243c/cbe1ebf3-0fd2-468b-b752-73c1c63eb76e/0e5af4fe-5ef2-4486-974c-49740f34623a"
-          (reference "#PWR0188") (unit 1)
+          (reference "#PWR0195") (unit 1)
         )
       )
@@
         )
         (path "/100bb8d1-c3d6-4e1f-87b6-72e4e187243c/cbe1ebf3-0fd2-468b-b752-73c1c63eb76e/0e5af4fe-5ef2-4486-974c-49740f34623a"
-          (reference "C53") (unit 1)
+          (reference "C57") (unit 1)
         )
       )
@@
         )
         (path "/100bb8d1-c3d6-4e1f-87b6-72e4e187243c/cbe1ebf3-0fd2-468b-b752-73c1c63eb76e/0e5af4fe-5ef2-4486-974c-49740f34623a"
-          (reference "#PWR0190") (unit 1)
+          (reference "#PWR0197") (unit 1)
         )
       )
@@
         )
         (path "/100bb8d1-c3d6-4e1f-87b6-72e4e187243c/cbe1ebf3-0fd2-468b-b752-73c1c63eb76e/0e5af4fe-5ef2-4486-974c-49740f34623a"
-          (reference "#PWR0186") (unit 1)
+          (reference "#PWR0193") (unit 1)
         )
       )
@@
   (symbol (lib_id "74xx:74HCT04") (at 257.81 38.1 0) (unit 7)
     (in_bom yes) (on_board yes) (dnp no) (fields_autoplaced)
-    (property "Reference" "U44" (at 264.16 36.83 0)
+    (property "Reference" "U46" (at 264.16 36.83 0)
       (effects (font (size 1.27 1.27)) (justify left))
     )
@@
       (project "8-bit-cpu"
         (path "/100bb8d1-c3d6-4e1f-87b6-72e4e187243c/cbe1ebf3-0fd2-468b-b752-73c1c63eb76e/0e5af4fe-5ef2-4486-974c-49740f34623a"
-          (reference "U44") (unit 7)
+          (reference "U46") (unit 7)
         )
       )
@@
   (symbol (lib_id "74xx:74HCT04") (at 73.66 134.62 180) (unit 4)
     (in_bom yes) (on_board yes) (dnp no) (fields_autoplaced)
-    (property "Reference" "U44" (at 73.66 125.73 0)
+    (property "Reference" "U46" (at 73.66 125.73 0)
       (effects (font (size 1.27 1.27)))
     )
@@
       (project "8-bit-cpu"
         (path "/100bb8d1-c3d6-4e1f-87b6-72e4e187243c/cbe1ebf3-0fd2-468b-b752-73c1c63eb76e/0e5af4fe-5ef2-4486-974c-49740f34623a"
-          (reference "U44") (unit 4)
+          (reference "U46") (unit 4)
         )
       )
@@
   (symbol (lib_id "74xx:74HCT04") (at 73.66 92.71 180) (unit 1)
     (in_bom yes) (on_board yes) (dnp no) (fields_autoplaced)
-    (property "Reference" "U44" (at 73.66 83.82 0)
+    (property "Reference" "U46" (at 73.66 83.82 0)
       (effects (font (size 1.27 1.27)))
     )
@@
       (project "8-bit-cpu"
         (path "/100bb8d1-c3d6-4e1f-87b6-72e4e187243c/cbe1ebf3-0fd2-468b-b752-73c1c63eb76e/0e5af4fe-5ef2-4486-974c-49740f34623a"
-          (reference "U44") (unit 1)
-        )
-      )
+          (reference "U46") (unit 1)
+        )
+      )

Commit message: kicad update
Parts:
- D81: renamed from D5; footprint LED_THT:LED_D5.0mm -> 01_my_library:LED_D5.0mm
- D82: renamed from D6; footprint LED_THT:LED_D5.0mm -> 01_my_library:LED_D5.0mm
- D83: renamed from D7; footprint LED_THT:LED_D5.0mm -> 01_my_library:LED_D5.0mm
- D84: renamed from D8; footprint LED_THT:LED_D5.0mm -> 01_my_library:LED_D5.0mm
- D85: renamed from D9; footprint LED_THT:LED_D5.0mm -> 01_my_library:LED_D5.0mm
- D86: renamed from D10; footprint LED_THT:LED_D5.0mm -> 01_my_library:LED_D5.0mm
- D87: renamed from D11; footprint LED_THT:LED_D5.0mm -> 01_my_library:LED_D5.0mm
- D88: renamed from D12; footprint LED_THT:LED_D5.0mm -> 01_my_library:LED_D5.0mm
- renumbered C4 to C60, C1 to C61, R11 to R125, R12 to R126, R13 to R127, R14 to R128, R15 to R129, R16 to R130, R17 to R131, R18 to R132, U37 to U47
