File: microstep-counter.kicad_sch (KiCad schematic)
At the start: 24 parts, among them U41 74HCT00, U44 74HCT138, U45 74HCT161

Commit message: kicad update
Parts:
- D72, D73, D74, D75, D76, D77, D78, D79, D80: footprint LED_THT:LED_D5.0mm -> 01_my_library:LED_D5.0mm
- renumbered C2 to C57, C2 to C58, C2 to C59
