File: middle-microcode-eeprom.kicad_sch (KiCad schematic)
At the start: 20 parts, among them U37 AT28C64B, U53 74HCT04

Commit message: add pdf for instructions
Other:
- company: (none) -> TBR Designs
- title: (none) -> 8-bit CPU
Changed lines of the file:
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@@
 (kicad_sch (version 20230121) (generator eeschema)
   (paper "A4")
+  (title_block
+    (title "8-bit CPU")
+    (date "2023-11-28")
+    (rev "1.0")
+    (company "TBR Designs")
+  )
   (junction (at 118.11 60.96) (diameter 0) (color 0 0 0 0)
   )

Commit message: add arduino headers for programming
Parts:
- U53: footprint (none) -> Package_DIP:DIP-14_W7.62mm
Changed lines of the file:
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@@
       (effects (font (size 1.27 1.27)) (justify left))
     )
-    (property "Footprint" "" (at 255.27 49.53 0)
+    (property "Footprint" "Package_DIP:DIP-14_W7.62mm" (at 255.27 49.53 0)
       (effects (font (size 1.27 1.27)) hide)
     )
@@
       (effects (font (size 1.27 1.27)))
     )
-    (property "Footprint" "" (at 71.12 132.08 0)
+    (property "Footprint" "Package_DIP:DIP-14_W7.62mm" (at 71.12 132.08 0)
       (effects (font (size 1.27 1.27)) hide)
     )
@@
       (effects (font (size 1.27 1.27)))
     )
-    (property "Footprint" "" (at 71.12 118.11 0)
+    (property "Footprint" "Package_DIP:DIP-14_W7.62mm" (at 71.12 118.11 0)
       (effects (font (size 1.27 1.27)) hide)
     )
@@
       (effects (font (size 1.27 1.27)))
     )
-    (property "Footprint" "" (at 71.12 104.14 0)
+    (property "Footprint" "Package_DIP:DIP-14_W7.62mm" (at 71.12 104.14 0)
       (effects (font (size 1.27 1.27)) hide)
     )
@@
       (effects (font (size 1.27 1.27)))
     )
-    (property "Footprint" "" (at 71.12 160.02 0)
+    (property "Footprint" "Package_DIP:DIP-14_W7.62mm" (at 71.12 160.02 0)
       (effects (font (size 1.27 1.27)) hide)
     )
@@
       (effects (font (size 1.27 1.27)))
     )
-    (property "Footprint" "" (at 71.12 173.99 0)
+    (property "Footprint" "Package_DIP:DIP-14_W7.62mm" (at 71.12 173.99 0)
       (effects (font (size 1.27 1.27)) hide)
     )
@@
       (effects (font (size 1.27 1.27)))
     )
-    (property "Footprint" "" (at 71.12 146.05 0)
-      (effects (font (size 1.27 1.27)) hide)
-    )
+    (property "Footprint" "Package_DIP:DIP-14_W7.62mm" (at 71.12 146.05 0)
+      (effects (font (size 1.27 1.27)) hide)
+    )

Commit message: cleanup
Parts:
- D10, D11, D12, D5, D6, D7, D8, D9: value YELLOW -> BLUE
Changed lines of the file:
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@@
       (effects (font (size 1.27 1.27)) (justify right))
     )
-    (property "Value" "YELLOW" (at 241.3 147.32 90)
+    (property "Value" "BLUE" (at 241.3 147.32 90)
       (effects (font (size 1.27 1.27)) (justify right))
     )
@@
       (effects (font (size 1.27 1.27)) (justify right))
     )
-    (property "Value" "YELLOW" (at 190.5 147.32 90)
+    (property "Value" "BLUE" (at 190.5 147.32 90)
       (effects (font (size 1.27 1.27)) (justify right))
     )
@@
         )
         (path "/100bb8d1-c3d6-4e1f-87b6-72e4e187243c/cbe1ebf3-0fd2-468b-b752-73c1c63eb76e/b110281f-f2a0-4921-be20-6dcbfc1964e6"
-          (reference "#PWR0189") (unit 1)
+          (reference "#PWR0192") (unit 1)
         )
       )
@@
         )
         (path "/100bb8d1-c3d6-4e1f-87b6-72e4e187243c/cbe1ebf3-0fd2-468b-b752-73c1c63eb76e/b110281f-f2a0-4921-be20-6dcbfc1964e6"
-          (reference "#PWR0194") (unit 1)
+          (reference "#PWR0197") (unit 1)
         )
       )
@@
         )
         (path "/100bb8d1-c3d6-4e1f-87b6-72e4e187243c/cbe1ebf3-0fd2-468b-b752-73c1c63eb76e/b110281f-f2a0-4921-be20-6dcbfc1964e6"
-          (reference "#PWR0190") (unit 1)
+          (reference "#PWR0193") (unit 1)
         )
       )
@@
         )
         (path "/100bb8d1-c3d6-4e1f-87b6-72e4e187243c/cbe1ebf3-0fd2-468b-b752-73c1c63eb76e/b110281f-f2a0-4921-be20-6dcbfc1964e6"
-          (reference "#PWR0193") (unit 1)
+          (reference "#PWR0196") (unit 1)
         )
       )
@@
         )
         (path "/100bb8d1-c3d6-4e1f-87b6-72e4e187243c/cbe1ebf3-0fd2-468b-b752-73c1c63eb76e/b110281f-f2a0-4921-be20-6dcbfc1964e6"
-          (reference "#PWR0191") (unit 1)
+          (reference "#PWR0194") (unit 1)
         )
       )
@@
       (effects (font (size 1.27 1.27)) (justify right))
     )
-    (property "Value" "YELLOW" (at 251.46 147.32 90)
+    (property "Value" "BLUE" (at 251.46 147.32 90)
       (effects (font (size 1.27 1.27)) (justify right))
     )
@@
       (effects (font (size 1.27 1.27)) (justify right))
     )
-    (property "Value" "YELLOW" (at 261.62 147.32 90)
+    (property "Value" "BLUE" (at 261.62 147.32 90)
       (effects (font (size 1.27 1.27)) (justify right))
     )
@@
         )
         (path "/100bb8d1-c3d6-4e1f-87b6-72e4e187243c/cbe1ebf3-0fd2-468b-b752-73c1c63eb76e/b110281f-f2a0-4921-be20-6dcbfc1964e6"
-          (reference "#PWR0195") (unit 1)
+          (reference "#PWR0198") (unit 1)
         )
       )
@@
       (effects (font (size 1.27 1.27)) (justify right))
     )
-    (property "Value" "YELLOW" (at 231.14 147.32 90)
+    (property "Value" "BLUE" (at 231.14 147.32 90)
       (effects (font (size 1.27 1.27)) (justify right))
     )
@@
       (effects (font (size 1.27 1.27)) (justify right))
     )
-    (property "Value" "YELLOW" (at 220.98 147.32 90)
+    (property "Value" "BLUE" (at 220.98 147.32 90)
       (effects (font (size 1.27 1.27)) (justify right))
     )
@@
       (effects (font (size 1.27 1.27)) (justify right))
     )
-    (property "Value" "YELLOW" (at 200.66 147.32 90)
+    (property "Value" "BLUE" (at 200.66 147.32 90)
       (effects (font (size 1.27 1.27)) (justify right))
     )
@@
       (effects (font (size 1.27 1.27)) (justify right))
     )
-    (property "Value" "YELLOW" (at 210.82 147.32 90)
+    (property "Value" "BLUE" (at 210.82 147.32 90)
       (effects (font (size 1.27 1.27)) (justify right))
     )
@@
         )
         (path "/100bb8d1-c3d6-4e1f-87b6-72e4e187243c/cbe1ebf3-0fd2-468b-b752-73c1c63eb76e/b110281f-f2a0-4921-be20-6dcbfc1964e6"
-          (reference "#PWR0192") (unit 1)
-        )
-      )
+          (reference "#PWR0195") (unit 1)
+        )
+      )

Commit message: trying to solve issues
Connections:
- net CARRY_FLAG renamed EEPROM_9
- net INSTRUCTION_0 renamed EEPROM_3
- net INSTRUCTION_1 renamed EEPROM_4
- net INSTRUCTION_2 renamed EEPROM_5
- net INSTRUCTION_3 renamed EEPROM_6
- net INSTRUCTION_4 renamed EEPROM_7
- net INSTRUCTION_5 renamed EEPROM_8
- net ZERO_FLAG renamed EEPROM_10
Changed lines of the file:
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@@
     (effects (font (size 1.27 1.27)) (justify left bottom))
   )
+  (hierarchical_label "EEPROM_3" (shape input) (at 39.37 36.83 180) (fields_autoplaced)
+    (effects (font (size 1.27 1.27)) (justify right))
+  )
+  (hierarchical_label "MS_2" (shape input) (at 39.37 34.29 180) (fields_autoplaced)
+    (effects (font (size 1.27 1.27)) (justify right))
+  )
+  (hierarchical_label "EEPROM_8" (shape input) (at 39.37 49.53 180) (fields_autoplaced)
+    (effects (font (size 1.27 1.27)) (justify right))
+  )
+  (hierarchical_label "MS_0" (shape input) (at 39.37 29.21 180) (fields_autoplaced)
+    (effects (font (size 1.27 1.27)) (justify right))
+  )
+  (hierarchical_label "HALT" (shape output) (at 39.37 92.71 180) (fields_autoplaced)
+    (effects (font (size 1.27 1.27)) (justify right))
+  )
+  (hierarchical_label "EEPROM_6" (shape input) (at 39.37 44.45 180) (fields_autoplaced)
+    (effects (font (size 1.27 1.27)) (justify right))
+  )
+  (hierarchical_label "SUBTRACT" (shape output) (at 39.37 90.17 180) (fields_autoplaced)
+    (effects (font (size 1.27 1.27)) (justify right))
+  )
+  (hierarchical_label "EEPROM_5" (shape input) (at 39.37 41.91 180) (fields_autoplaced)
+    (effects (font (size 1.27 1.27)) (justify right))
+  )
+  (hierarchical_label "~{FLAGS_INPUT}" (shape output) (at 39.37 107.95 180) (fields_autoplaced)
+    (effects (font (size 1.27 1.27)) (justify right))
+  )
+  (hierarchical_label "~{B_INPUT}" (shape output) (at 39.37 100.33 180) (fields_autoplaced)
+    (effects (font (size 1.27 1.27)) (justify right))
+  )
+  (hierarchical_label "EEPROM_7" (shape input) (at 39.37 46.99 180) (fields_autoplaced)
+    (effects (font (size 1.27 1.27)) (justify right))
+  )
+  (hierarchical_label "EEPROM_9" (shape input) (at 39.37 52.07 180) (fields_autoplaced)
+    (effects (font (size 1.27 1.27)) (justify right))
+  )
+  (hierarchical_label "~{OUTPUT_INPUT}" (shape output) (at 39.37 105.41 180) (fields_autoplaced)
+    (effects (font (size 1.27 1.27)) (justify right))
+  )
+  (hierarchical_label "~{ALU_OUTPUT}" (shape output) (at 39.37 97.79 180) (fields_autoplaced)
+    (effects (font (size 1.27 1.27)) (justify right))
+  )
   (hierarchical_label "MS_1" (shape input) (at 39.37 31.75 180) (fields_autoplaced)
     (effects (font (size 1.27 1.27)) (justify right))
   )
-  (hierarchical_label "INSTRUCTION_3" (shape input) (at 39.37 44.45 180) (fields_autoplaced)
-    (effects (font (size 1.27 1.27)) (justify right))
-  )
-  (hierarchical_label "INSTRUCTION_1" (shape input) (at 39.37 39.37 180) (fields_autoplaced)
-    (effects (font (size 1.27 1.27)) (justify right))
-  )
-  (hierarchical_label "ZERO_FLAG" (shape input) (at 39.37 54.61 180) (fields_autoplaced)
-    (effects (font (size 1.27 1.27)) (justify right))
-  )
-  (hierarchical_label "CARRY_FLAG" (shape input) (at 39.37 52.07 180) (fields_autoplaced)
-    (effects (font (size 1.27 1.27)) (justify right))
-  )
-  (hierarchical_label "MS_2" (shape input) (at 39.37 34.29 180) (fields_autoplaced)
-    (effects (font (size 1.27 1.27)) (justify right))
-  )
-  (hierarchical_label "INSTRUCTION_5" (shape input) (at 39.37 49.53 180) (fields_autoplaced)
-    (effects (font (size 1.27 1.27)) (justify right))
-  )
-  (hierarchical_label "HALT" (shape output) (at 39.37 92.71 180) (fields_autoplaced)
-    (effects (font (size 1.27 1.27)) (justify right))
-  )
-  (hierarchical_label "INSTRUCTION_4" (shape input) (at 39.37 46.99 180) (fields_autoplaced)
-    (effects (font (size 1.27 1.27)) (justify right))
-  )
-  (hierarchical_label "INSTRUCTION_2" (shape input) (at 39.37 41.91 180) (fields_autoplaced)
-    (effects (font (size 1.27 1.27)) (justify right))
-  )
-  (hierarchical_label "SUBTRACT" (shape output) (at 39.37 90.17 180) (fields_autoplaced)
-    (effects (font (size 1.27 1.27)) (justify right))
-  )
-  (hierarchical_label "~{FLAGS_INPUT}" (shape output) (at 39.37 107.95 180) (fields_autoplaced)
-    (effects (font (size 1.27 1.27)) (justify right))
-  )
-  (hierarchical_label "~{B_INPUT}" (shape output) (at 39.37 100.33 180) (fields_autoplaced)
-    (effects (font (size 1.27 1.27)) (justify right))
-  )
-  (hierarchical_label "~{OUTPUT_INPUT}" (shape output) (at 39.37 105.41 180) (fields_autoplaced)
-    (effects (font (size 1.27 1.27)) (justify right))
-  )
-  (hierarchical_label "~{ALU_OUTPUT}" (shape output) (at 39.37 97.79 180) (fields_autoplaced)
-    (effects (font (size 1.27 1.27)) (justify right))
-  )
-  (hierarchical_label "MS_0" (shape input) (at 39.37 29.21 180) (fields_autoplaced)
+  (hierarchical_label "EEPROM_10" (shape input) (at 39.37 54.61 180) (fields_autoplaced)
     (effects (font (size 1.27 1.27)) (justify right))
   )
@@
     (effects (font (size 1.27 1.27)) (justify right))
   )
-  (hierarchical_label "INSTRUCTION_0" (shape input) (at 39.37 36.83 180) (fields_autoplaced)
+  (hierarchical_label "EEPROM_4" (shape input) (at 39.37 39.37 180) (fields_autoplaced)
     (effects (font (size 1.27 1.27)) (justify right))
   )
@@
         )
         (path "/100bb8d1-c3d6-4e1f-87b6-72e4e187243c/cbe1ebf3-0fd2-468b-b752-73c1c63eb76e/b110281f-f2a0-4921-be20-6dcbfc1964e6"
-          (reference "U46") (unit 7)
+          (reference "U48") (unit 7)
         )
       )
@@
         )
         (path "/100bb8d1-c3d6-4e1f-87b6-72e4e187243c/cbe1ebf3-0fd2-468b-b752-73c1c63eb76e/b110281f-f2a0-4921-be20-6dcbfc1964e6"
-          (reference "#PWR0192") (unit 1)
+          (reference "#PWR0199") (unit 1)
         )
       )
@@
         )
         (path "/100bb8d1-c3d6-4e1f-87b6-72e4e187243c/cbe1ebf3-0fd2-468b-b752-73c1c63eb76e/b110281f-f2a0-4921-be20-6dcbfc1964e6"
-          (reference "#PWR0197") (unit 1)
+          (reference "#PWR0204") (unit 1)
         )
       )
@@
         )
         (path "/100bb8d1-c3d6-4e1f-87b6-72e4e187243c/cbe1ebf3-0fd2-468b-b752-73c1c63eb76e/b110281f-f2a0-4921-be20-6dcbfc1964e6"
-          (reference "U47") (unit 1)
+          (reference "U49") (unit 1)
         )
       )
@@
         )
         (path "/100bb8d1-c3d6-4e1f-87b6-72e4e187243c/cbe1ebf3-0fd2-468b-b752-73c1c63eb76e/b110281f-f2a0-4921-be20-6dcbfc1964e6"
-          (reference "#PWR0193") (unit 1)
+          (reference "#PWR0200") (unit 1)
         )
       )
@@
         )
         (path "/100bb8d1-c3d6-4e1f-87b6-72e4e187243c/cbe1ebf3-0fd2-468b-b752-73c1c63eb76e/b110281f-f2a0-4921-be20-6dcbfc1964e6"
-          (reference "U46") (unit 3)
+          (reference "U48") (unit 3)
         )
       )
@@
         )
         (path "/100bb8d1-c3d6-4e1f-87b6-72e4e187243c/cbe1ebf3-0fd2-468b-b752-73c1c63eb76e/b110281f-f2a0-4921-be20-6dcbfc1964e6"
-          (reference "#PWR0196") (unit 1)
+          (reference "#PWR0203") (unit 1)
         )
       )
@@
         )
         (path "/100bb8d1-c3d6-4e1f-87b6-72e4e187243c/cbe1ebf3-0fd2-468b-b752-73c1c63eb76e/b110281f-f2a0-4921-be20-6dcbfc1964e6"
-          (reference "#PWR0194") (unit 1)
+          (reference "#PWR0201") (unit 1)
         )
       )
@@
         )
         (path "/100bb8d1-c3d6-4e1f-87b6-72e4e187243c/cbe1ebf3-0fd2-468b-b752-73c1c63eb76e/b110281f-f2a0-4921-be20-6dcbfc1964e6"
-          (reference "#PWR0198") (unit 1)
+          (reference "#PWR0205") (unit 1)
         )
       )
@@
         )
         (path "/100bb8d1-c3d6-4e1f-87b6-72e4e187243c/cbe1ebf3-0fd2-468b-b752-73c1c63eb76e/b110281f-f2a0-4921-be20-6dcbfc1964e6"
-          (reference "U46") (unit 2)
+          (reference "U48") (unit 2)
         )
       )
@@
         )
         (path "/100bb8d1-c3d6-4e1f-87b6-72e4e187243c/cbe1ebf3-0fd2-468b-b752-73c1c63eb76e/b110281f-f2a0-4921-be20-6dcbfc1964e6"
-          (reference "U46") (unit 1)
+          (reference "U48") (unit 1)
         )
       )
@@
         )
         (path "/100bb8d1-c3d6-4e1f-87b6-72e4e187243c/cbe1ebf3-0fd2-468b-b752-73c1c63eb76e/b110281f-f2a0-4921-be20-6dcbfc1964e6"
-          (reference "C54") (unit 1)
+          (reference "C58") (unit 1)
         )
       )
@@
         )
         (path "/100bb8d1-c3d6-4e1f-87b6-72e4e187243c/cbe1ebf3-0fd2-468b-b752-73c1c63eb76e/b110281f-f2a0-4921-be20-6dcbfc1964e6"
-          (reference "U46") (unit 5)
+          (reference "U48") (unit 5)
         )
       )
@@
         )
         (path "/100bb8d1-c3d6-4e1f-87b6-72e4e187243c/cbe1ebf3-0fd2-468b-b752-73c1c63eb76e/b110281f-f2a0-4921-be20-6dcbfc1964e6"
-          (reference "U46") (unit 6)
+          (reference "U48") (unit 6)
         )
       )
@@
         )
         (path "/100bb8d1-c3d6-4e1f-87b6-72e4e187243c/cbe1ebf3-0fd2-468b-b752-73c1c63eb76e/b110281f-f2a0-4921-be20-6dcbfc1964e6"
-          (reference "U46") (unit 4)
+          (reference "U48") (unit 4)
         )
       )
@@
         )
         (path "/100bb8d1-c3d6-4e1f-87b6-72e4e187243c/cbe1ebf3-0fd2-468b-b752-73c1c63eb76e/b110281f-f2a0-4921-be20-6dcbfc1964e6"
-          (reference "C55") (unit 1)
+          (reference "C59") (unit 1)
         )
       )
@@
         )
         (path "/100bb8d1-c3d6-4e1f-87b6-72e4e187243c/cbe1ebf3-0fd2-468b-b752-73c1c63eb76e/b110281f-f2a0-4921-be20-6dcbfc1964e6"
-          (reference "#PWR0195") (unit 1)
-        )
-      )
+          (reference "#PWR0202") (unit 1)
+        )
+      )

Commit message: kicad update
Parts:
- D89: renamed from D5; footprint LED_THT:LED_D5.0mm -> 01_my_library:LED_D5.0mm
- D90: renamed from D6; footprint LED_THT:LED_D5.0mm -> 01_my_library:LED_D5.0mm
- D91: renamed from D7; footprint LED_THT:LED_D5.0mm -> 01_my_library:LED_D5.0mm
- D92: renamed from D8; footprint LED_THT:LED_D5.0mm -> 01_my_library:LED_D5.0mm
- D93: renamed from D9; footprint LED_THT:LED_D5.0mm -> 01_my_library:LED_D5.0mm
- D94: renamed from D10; footprint LED_THT:LED_D5.0mm -> 01_my_library:LED_D5.0mm
- D95: renamed from D11; footprint LED_THT:LED_D5.0mm -> 01_my_library:LED_D5.0mm
- D96: renamed from D12; footprint LED_THT:LED_D5.0mm -> 01_my_library:LED_D5.0mm
- renumbered C4 to C62, C1 to C63, R11 to R133, R12 to R134, R13 to R135, R14 to R136, R15 to R137, R16 to R138, R17 to R139, R18 to R140, U53 to U48, U37 to U49
