File: output.kicad_sch (KiCad schematic)
At the start: 28 parts, among them J4 2_Complement_Header, U32 74HCT107, U33 74HCT139, U35 LTC-5723HR, U37 AT28C64B, U4 LMC555xN, U8 74HCT173, U9 74HCT173

Commit message: some more layout
Connections:
- net +5V: now also C1.1, C1.1, U32.14 (VCC), U33.16 (VCC)
Changed lines of the file:
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@@
   (junction (at 119.38 152.4) (diameter 0) (color 0 0 0 0)
   )
+  (junction (at 262.89 20.32) (diameter 0) (color 0 0 0 0)
+  )
   (junction (at 113.03 58.42) (diameter 0) (color 0 0 0 0)
   )
@@
   )
   (junction (at 119.38 140.97) (diameter 0) (color 0 0 0 0)
+  )
+  (junction (at 237.49 20.32) (diameter 0) (color 0 0 0 0)
   )
   (junction (at 127 163.83) (diameter 0) (color 0 0 0 0)
@@
     )
   )
+  (symbol (lib_id "power:+5V") (at 262.89 20.32 0) (unit 1)
+    (in_bom yes) (on_board yes) (dnp no) (fields_autoplaced)
+    (property "Reference" "#PWR0272" (at 262.89 24.13 0)
+      (effects (font (size 1.27 1.27)) hide)
+    )
+    (property "Value" "+5V" (at 262.89 15.24 0)
+      (effects (font (size 1.27 1.27)))
+    )
+    (property "Footprint" "" (at 262.89 20.32 0)
+      (effects (font (size 1.27 1.27)) hide)
+    )
+    (property "Datasheet" "" (at 262.89 20.32 0)
+      (effects (font (size 1.27 1.27)) hide)
+    )
+    (pin "1")
+    (instances
+      (project "8-bit-cpu"
+        (path "/100bb8d1-c3d6-4e1f-87b6-72e4e187243c/2c3402b7-c2ba-43ce-9f44-0fa5e5dc9ef7"
+          (reference "#PWR0272") (unit 1)
+        )
+      )
+    )
+  )
   (symbol (lib_id "Device:C") (at 90.17 87.63 0) (unit 1)
     (in_bom yes) (on_board yes) (dnp no)
@@
         )
       )
+    )
+  )
+  (symbol (lib_id "power:+5V") (at 237.49 20.32 0) (unit 1)
+    (in_bom yes) (on_board yes) (dnp no) (fields_autoplaced)
+    (property "Reference" "#PWR0271" (at 237.49 24.13 0)
+      (effects (font (size 1.27 1.27)) hide)
+    )
+    (property "Value" "+5V" (at 237.49 15.24 0)
+      (effects (font (size 1.27 1.27)))
+    )
+    (property "Footprint" "" (at 237.49 20.32 0)
+      (effects (font (size 1.27 1.27)) hide)
+    )
+    (property "Datasheet" "" (at 237.49 20.32 0)
+      (effects (font (size 1.27 1.27)) hide)
+    )
+    (pin "1")
+    (instances
+      (project "8-bit-cpu"
+        (path "/100bb8d1-c3d6-4e1f-87b6-72e4e187243c/2c3402b7-c2ba-43ce-9f44-0fa5e5dc9ef7"
+          (reference "#PWR0271") (unit 1)
+        )
+      )

Commit message: kicad update
Parts:
- renumbered C1 to C42, C1 to C43, C1 to C44, C5 to C45, C6 to C46, C1 to C47, C1 to C48, C1 to C49, C13 to C50, R18 to R96, R19 to R97, U4 to U34, U8 to U36, U9 to U38
