File: program-counter.kicad_sch (KiCad schematic)
At the start: 22 parts, among them U30 74HCT161, U31 74HCT161, U7 74HCT245

Commit message: changed symbols
Parts:
- U30, U31: symbol 74xx:74LS161 -> 01_my_library:74HCT161
- U7: symbol 74xx:74HC245 -> 01_my_library:74HCT245
Changed lines of the file:
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@@
     )
   )
-  (symbol (lib_id "74xx:74LS161") (at 151.13 83.82 270) (unit 1)
+  (symbol (lib_id "01_my_library:74HCT161") (at 151.13 83.82 270) (unit 1)
     (in_bom yes) (on_board yes) (dnp no)
     (property "Reference" "U30" (at 137.16 96.52 90)
@@
       (effects (font (size 1.27 1.27)) hide)
     )
-    (property "Datasheet" "http://www.ti.com/lit/gpn/sn74LS161" (at 151.13 83.82 0)
+    (property "Datasheet" "https://www.ti.com/lit/ds/symlink/cd54hct163.pdf?HQS=dis-mous-null-mousermode-dsf-pf-null-wwe&ts=1702794645288&ref_url=https%253A%252F%252Fwww.mouser.be%252F" (at 125.73 83.82 0)
       (effects (font (size 1.27 1.27)) hide)
     )
@@
     )
   )
-  (symbol (lib_id "74xx:74LS161") (at 205.74 83.82 270) (unit 1)
+  (symbol (lib_id "01_my_library:74HCT161") (at 205.74 83.82 270) (unit 1)
     (in_bom yes) (on_board yes) (dnp no)
     (property "Reference" "U31" (at 191.77 96.52 90)
@@
       (effects (font (size 1.27 1.27)) hide)
     )
-    (property "Datasheet" "http://www.ti.com/lit/gpn/sn74LS161" (at 205.74 83.82 0)
+    (property "Datasheet" "https://www.ti.com/lit/ds/symlink/cd54hct163.pdf?HQS=dis-mous-null-mousermode-dsf-pf-null-wwe&ts=1702794645288&ref_url=https%253A%252F%252Fwww.mouser.be%252F" (at 180.34 83.82 0)
       (effects (font (size 1.27 1.27)) hide)
     )
@@
     )
   )
-  (symbol (lib_id "74xx:74HC245") (at 77.47 83.82 270) (unit 1)
+  (symbol (lib_id "01_my_library:74HCT245") (at 77.47 83.82 270) (unit 1)
     (in_bom yes) (on_board yes) (dnp no)
     (property "Reference" "U7" (at 63.5 96.52 90)
@@
       (effects (font (size 1.27 1.27)) hide)
     )
-    (property "Datasheet" "http://www.ti.com/lit/gpn/sn74HC245" (at 77.47 83.82 0)
-      (effects (font (size 1.27 1.27)) hide)
-    )
+    (property "Datasheet" "https://www.ti.com/lit/ds/symlink/sn74hct245.pdf?ts=1702763405638&ref_url=https%253A%252F%252Fwww.google.com%252F" (at 54.61 83.82 0)
+      (effects (font (size 1.27 1.27)) hide)
+    )

Commit message: readme
Parts:
- added C13: 10n, 01_my_library:C_Disc_D4.0mm_W2.6mm_P2.50mm, symbol Device:C
Connections:
- net GND: now also C13.2
- net ~{RESET}: now also C13.1
Changed lines of the file:
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@@
   (junction (at 57.15 83.82) (diameter 0) (color 0 0 0 0)
+  )
+  (junction (at 193.04 63.5) (diameter 0) (color 255 0 0 1)
   )
   (junction (at 78.74 125.73) (diameter 0) (color 0 0 0 0)
@@
     (stroke (width 0) (type default) (color 255 0 0 1))
   )
+  (wire (pts (xy 193.04 39.37) (xy 200.66 39.37))
+    (stroke (width 0) (type default) (color 255 0 0 1))
+  )
   (wire (pts (xy 161.29 39.37) (xy 77.47 39.37))
     (stroke (width 0) (type default) (color 0 0 255 1))
@@
     (stroke (width 0) (type default) (color 0 0 255 1))
   )
+  (wire (pts (xy 200.66 39.37) (xy 200.66 41.91))
+    (stroke (width 0) (type default) (color 255 0 0 1))
+  )
   (wire (pts (xy 119.38 160.02) (xy 129.54 160.02))
     (stroke (width 0) (type default))
@@
   (wire (pts (xy 34.29 29.21) (xy 87.63 29.21))
     (stroke (width 0) (type default) (color 0 0 255 1))
+  )
+  (wire (pts (xy 193.04 63.5) (xy 193.04 39.37))
+    (stroke (width 0) (type default) (color 255 0 0 1))
   )
   (wire (pts (xy 34.29 58.42) (xy 148.59 58.42))
@@
     )
   )
+  (symbol (lib_id "Device:C") (at 200.66 45.72 0) (unit 1)
+    (in_bom yes) (on_board yes) (dnp yes) (fields_autoplaced)
+    (property "Reference" "C13" (at 204.47 44.45 0)
+      (effects (font (size 1.27 1.27)) (justify left))
+    )
+    (property "Value" "10n" (at 204.47 46.99 0)
+      (effects (font (size 1.27 1.27)) (justify left))
+    )
+    (property "Footprint" "01_my_library:C_Disc_D4.0mm_W2.6mm_P2.50mm" (at 201.6252 49.53 0)
+      (effects (font (size 1.27 1.27)) hide)
+    )
+    (property "Datasheet" "~" (at 200.66 45.72 0)
+      (effects (font (size 1.27 1.27)) hide)
+    )
+    (pin "1")
+    (pin "2")
+    (instances
+      (project "8-bit-cpu"
+        (path "/100bb8d1-c3d6-4e1f-87b6-72e4e187243c/651dfbaf-e340-4976-8216-793c5a5aaa3b"
+          (reference "C13") (unit 1)
+        )
+        (path "/100bb8d1-c3d6-4e1f-87b6-72e4e187243c/eeec1d6e-c04a-42fe-8103-cb8adc13344c"
+          (reference "C77") (unit 1)
+        )
+      )
+    )
+  )
   (symbol (lib_id "power:GND") (at 231.14 91.44 0) (unit 1)
     (in_bom yes) (on_board yes) (dnp no) (fields_autoplaced)
@@
         )
       )
+    )
+  )
+  (symbol (lib_id "power:GND") (at 200.66 49.53 0) (unit 1)
+    (in_bom yes) (on_board yes) (dnp no) (fields_autoplaced)
+    (property "Reference" "#PWR03" (at 200.66 55.88 0)
+      (effects (font (size 1.27 1.27)) hide)
+    )
+    (property "Value" "GND" (at 200.66 54.61 0)
+      (effects (font (size 1.27 1.27)) hide)
+    )
+    (property "Footprint" "" (at 200.66 49.53 0)
+      (effects (font (size 1.27 1.27)) hide)
+    )
+    (property "Datasheet" "" (at 200.66 49.53 0)
+      (effects (font (size 1.27 1.27)) hide)
+    )
+    (pin "1")
+    (instances
+      (project "8-bit-cpu"
+        (path "/100bb8d1-c3d6-4e1f-87b6-72e4e187243c/45eb39c3-c748-461e-8330-08aae1247dee"
+          (reference "#PWR03") (unit 1)
+        )
+        (path "/100bb8d1-c3d6-4e1f-87b6-72e4e187243c/651dfbaf-e340-4976-8216-793c5a5aaa3b"
+          (reference "#PWR038") (unit 1)
+        )
+        (path "/100bb8d1-c3d6-4e1f-87b6-72e4e187243c/3568514a-e420-48fa-9fd5-7a290120765b"
+          (reference "#PWR056") (unit 1)
+        )
+        (path "/100bb8d1-c3d6-4e1f-87b6-72e4e187243c/eeec1d6e-c04a-42fe-8103-cb8adc13344c"
+          (reference "#PWR0265") (unit 1)
+        )
+      )

Commit message: kicad update
Parts:
- D56: renamed from D5; footprint LED_THT:LED_D5.0mm -> 01_my_library:LED_D5.0mm
- D57: renamed from D6; footprint LED_THT:LED_D5.0mm -> 01_my_library:LED_D5.0mm
- D58: renamed from D7; footprint LED_THT:LED_D5.0mm -> 01_my_library:LED_D5.0mm
- D59: renamed from D8; footprint LED_THT:LED_D5.0mm -> 01_my_library:LED_D5.0mm
- D60: renamed from D9; footprint LED_THT:LED_D5.0mm -> 01_my_library:LED_D5.0mm
- D61: renamed from D10; footprint LED_THT:LED_D5.0mm -> 01_my_library:LED_D5.0mm
- D62: renamed from D11; footprint LED_THT:LED_D5.0mm -> 01_my_library:LED_D5.0mm
- D63: renamed from D12; footprint LED_THT:LED_D5.0mm -> 01_my_library:LED_D5.0mm
- renumbered C13 to C38, C1 to C39, C1 to C40, C1 to C41, R11 to R88, R12 to R89, R13 to R90, R14 to R91, R15 to R92, R16 to R93, R17 to R94, R18 to R95, U7 to U29
