File: ram-address.kicad_sch (KiCad schematic)
At the start: 37 parts, among them J1 Arduino_Address_Programming_H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, SW3 SW_DIP_x08, U22 74HCT157, U23 74HCT157, U8 74HCT173, U9 74HCT173

Commit message: regenerated BOM
Parts:
- C27: footprint (none) -> 01_my_library:C_Disc_D4.0mm_W2.6mm_P2.50mm
Changed lines of the file:
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@@
       (effects (font (size 1.27 1.27)) (justify left))
     )
-    (property "Footprint" "" (at 145.7452 53.34 0)
+    (property "Footprint" "01_my_library:C_Disc_D4.0mm_W2.6mm_P2.50mm" (at 145.7452 53.34 0)
       (effects (font (size 1.27 1.27)) hide)
     )

Commit message: some more layout
Parts:
- renumbered C27 to C28
Changed lines of the file:
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@@
         )
         (path "/100bb8d1-c3d6-4e1f-87b6-72e4e187243c/33b906b8-f63f-4a46-8ef2-4150917936b8/b8600875-f531-45d3-8c06-c8d636c0c136"
-          (reference "#PWR0102") (unit 1)
+          (reference "#PWR0103") (unit 1)
         )
       )
@@
         )
         (path "/100bb8d1-c3d6-4e1f-87b6-72e4e187243c/33b906b8-f63f-4a46-8ef2-4150917936b8/b8600875-f531-45d3-8c06-c8d636c0c136"
-          (reference "#PWR090") (unit 1)
+          (reference "#PWR091") (unit 1)
         )
       )
@@
   (symbol (lib_id "power:GND") (at 46.99 138.43 0) (unit 1)
     (in_bom yes) (on_board yes) (dnp no) (fields_autoplaced)
-    (property "Reference" "#PWR099" (at 46.99 144.78 0)
+    (property "Reference" "#PWR0100" (at 46.99 144.78 0)
       (effects (font (size 1.27 1.27)) hide)
     )
@@
       (project "8-bit-cpu"
         (path "/100bb8d1-c3d6-4e1f-87b6-72e4e187243c/33b906b8-f63f-4a46-8ef2-4150917936b8/b8600875-f531-45d3-8c06-c8d636c0c136"
-          (reference "#PWR099") (unit 1)
+          (reference "#PWR0100") (unit 1)
         )
       )
@@
   (symbol (lib_id "power:GND") (at 144.78 69.85 0) (unit 1)
     (in_bom yes) (on_board yes) (dnp no) (fields_autoplaced)
-    (property "Reference" "#PWR092" (at 144.78 76.2 0)
+    (property "Reference" "#PWR093" (at 144.78 76.2 0)
       (effects (font (size 1.27 1.27)) hide)
     )
@@
       (project "8-bit-cpu"
         (path "/100bb8d1-c3d6-4e1f-87b6-72e4e187243c/33b906b8-f63f-4a46-8ef2-4150917936b8/b8600875-f531-45d3-8c06-c8d636c0c136"
-          (reference "#PWR092") (unit 1)
+          (reference "#PWR093") (unit 1)
         )
       )
@@
         )
         (path "/100bb8d1-c3d6-4e1f-87b6-72e4e187243c/33b906b8-f63f-4a46-8ef2-4150917936b8/b8600875-f531-45d3-8c06-c8d636c0c136"
-          (reference "#PWR095") (unit 1)
+          (reference "#PWR096") (unit 1)
         )
       )
@@
         )
         (path "/100bb8d1-c3d6-4e1f-87b6-72e4e187243c/33b906b8-f63f-4a46-8ef2-4150917936b8/b8600875-f531-45d3-8c06-c8d636c0c136"
-          (reference "C28") (unit 1)
+          (reference "C29") (unit 1)
         )
       )
@@
         )
         (path "/100bb8d1-c3d6-4e1f-87b6-72e4e187243c/33b906b8-f63f-4a46-8ef2-4150917936b8/b8600875-f531-45d3-8c06-c8d636c0c136"
-          (reference "#PWR094") (unit 1)
+          (reference "#PWR095") (unit 1)
         )
       )
@@
         )
         (path "/100bb8d1-c3d6-4e1f-87b6-72e4e187243c/33b906b8-f63f-4a46-8ef2-4150917936b8/b8600875-f531-45d3-8c06-c8d636c0c136"
-          (reference "#PWR091") (unit 1)
+          (reference "#PWR092") (unit 1)
         )
       )
@@
         )
         (path "/100bb8d1-c3d6-4e1f-87b6-72e4e187243c/33b906b8-f63f-4a46-8ef2-4150917936b8/b8600875-f531-45d3-8c06-c8d636c0c136"
-          (reference "#PWR098") (unit 1)
+          (reference "#PWR099") (unit 1)
         )
       )
@@
   (symbol (lib_id "power:GND") (at 31.75 64.77 0) (unit 1)
     (in_bom yes) (on_board yes) (dnp no) (fields_autoplaced)
-    (property "Reference" "#PWR089" (at 31.75 71.12 0)
+    (property "Reference" "#PWR090" (at 31.75 71.12 0)
       (effects (font (size 1.27 1.27)) hide)
     )
@@
       (project "8-bit-cpu"
         (path "/100bb8d1-c3d6-4e1f-87b6-72e4e187243c/33b906b8-f63f-4a46-8ef2-4150917936b8/b8600875-f531-45d3-8c06-c8d636c0c136"
-          (reference "#PWR089") (unit 1)
+          (reference "#PWR090") (unit 1)
         )
       )
@@
         )
         (path "/100bb8d1-c3d6-4e1f-87b6-72e4e187243c/33b906b8-f63f-4a46-8ef2-4150917936b8/b8600875-f531-45d3-8c06-c8d636c0c136"
-          (reference "#PWR0103") (unit 1)
+          (reference "#PWR0104") (unit 1)
         )
       )
@@
         )
         (path "/100bb8d1-c3d6-4e1f-87b6-72e4e187243c/33b906b8-f63f-4a46-8ef2-4150917936b8/b8600875-f531-45d3-8c06-c8d636c0c136"
-          (reference "C31") (unit 1)
+          (reference "C32") (unit 1)
         )
       )
@@
         )
         (path "/100bb8d1-c3d6-4e1f-87b6-72e4e187243c/33b906b8-f63f-4a46-8ef2-4150917936b8/b8600875-f531-45d3-8c06-c8d636c0c136"
-          (reference "C30") (unit 1)
+          (reference "C31") (unit 1)
         )
       )
@@
   (symbol (lib_id "power:GND") (at 111.76 138.43 0) (unit 1)
     (in_bom yes) (on_board yes) (dnp no) (fields_autoplaced)
-    (property "Reference" "#PWR0100" (at 111.76 144.78 0)
+    (property "Reference" "#PWR0101" (at 111.76 144.78 0)
       (effects (font (size 1.27 1.27)) hide)
     )
@@
       (project "8-bit-cpu"
         (path "/100bb8d1-c3d6-4e1f-87b6-72e4e187243c/33b906b8-f63f-4a46-8ef2-4150917936b8/b8600875-f531-45d3-8c06-c8d636c0c136"
-          (reference "#PWR0100") (unit 1)
+          (reference "#PWR0101") (unit 1)
         )
       )
@@
   (symbol (lib_id "Device:C") (at 144.78 49.53 0) (unit 1)
     (in_bom yes) (on_board yes) (dnp yes)
-    (property "Reference" "C27" (at 137.16 48.26 0)
+    (property "Reference" "C28" (at 137.16 48.26 0)
       (effects (font (size 1.27 1.27)) (justify left))
     )
@@
       (project "8-bit-cpu"
         (path "/100bb8d1-c3d6-4e1f-87b6-72e4e187243c/33b906b8-f63f-4a46-8ef2-4150917936b8/b8600875-f531-45d3-8c06-c8d636c0c136"
-          (reference "C27") (unit 1)
+          (reference "C28") (unit 1)
         )
       )
@@
   (symbol (lib_id "power:GND") (at 25.4 105.41 0) (unit 1)
     (in_bom yes) (on_board yes) (dnp no) (fields_autoplaced)
-    (property "Reference" "#PWR096" (at 25.4 111.76 0)
+    (property "Reference" "#PWR097" (at 25.4 111.76 0)
       (effects (font (size 1.27 1.27)) hide)
     )
@@
       (project "8-bit-cpu"
         (path "/100bb8d1-c3d6-4e1f-87b6-72e4e187243c/33b906b8-f63f-4a46-8ef2-4150917936b8/b8600875-f531-45d3-8c06-c8d636c0c136"
-          (reference "#PWR096") (unit 1)
+          (reference "#PWR097") (unit 1)
         )
       )
@@
         )
         (path "/100bb8d1-c3d6-4e1f-87b6-72e4e187243c/33b906b8-f63f-4a46-8ef2-4150917936b8/b8600875-f531-45d3-8c06-c8d636c0c136"
-          (reference "#PWR097") (unit 1)
+          (reference "#PWR098") (unit 1)
         )
       )
@@
         )
         (path "/100bb8d1-c3d6-4e1f-87b6-72e4e187243c/33b906b8-f63f-4a46-8ef2-4150917936b8/b8600875-f531-45d3-8c06-c8d636c0c136"
-          (reference "#PWR0101") (unit 1)
+          (reference "#PWR0102") (unit 1)
         )
       )
@@
   (symbol (lib_id "power:GND") (at 207.01 69.85 0) (unit 1)
     (in_bom yes) (on_board yes) (dnp no) (fields_autoplaced)
-    (property "Reference" "#PWR093" (at 207.01 76.2 0)
+    (property "Reference" "#PWR094" (at 207.01 76.2 0)
       (effects (font (size 1.27 1.27)) hide)
     )
@@
       (project "8-bit-cpu"
         (path "/100bb8d1-c3d6-4e1f-87b6-72e4e187243c/33b906b8-f63f-4a46-8ef2-4150917936b8/b8600875-f531-45d3-8c06-c8d636c0c136"
-          (reference "#PWR093") (unit 1)
+          (reference "#PWR094") (unit 1)
         )
       )
@@
         )
         (path "/100bb8d1-c3d6-4e1f-87b6-72e4e187243c/33b906b8-f63f-4a46-8ef2-4150917936b8/b8600875-f531-45d3-8c06-c8d636c0c136"
-          (reference "#PWR088") (unit 1)
+          (reference "#PWR089") (unit 1)
         )
       )
@@
         )
         (path "/100bb8d1-c3d6-4e1f-87b6-72e4e187243c/33b906b8-f63f-4a46-8ef2-4150917936b8/b8600875-f531-45d3-8c06-c8d636c0c136"
-          (reference "C29") (unit 1)
-        )
-      )
+          (reference "C30") (unit 1)
+        )
+      )

Commit message: kicad update
Parts:
- D45, D46: renamed from D5; footprint LED_THT:LED_D5.0mm -> 01_my_library:LED_D5.0mm
- D47: renamed from D6; footprint LED_THT:LED_D5.0mm -> 01_my_library:LED_D5.0mm
- D48: renamed from D7; footprint LED_THT:LED_D5.0mm -> 01_my_library:LED_D5.0mm
- D49: renamed from D8; footprint LED_THT:LED_D5.0mm -> 01_my_library:LED_D5.0mm
- D50: renamed from D9; footprint LED_THT:LED_D5.0mm -> 01_my_library:LED_D5.0mm
- D51: renamed from D10; footprint LED_THT:LED_D5.0mm -> 01_my_library:LED_D5.0mm
- D52: renamed from D11; footprint LED_THT:LED_D5.0mm -> 01_my_library:LED_D5.0mm
- D53: renamed from D12; footprint LED_THT:LED_D5.0mm -> 01_my_library:LED_D5.0mm
- renumbered C1 to C29, C1 to C30, C1 to C31, C1 to C32, R11 to R67, R11 to R68, R12 to R69, R13 to R70, R14 to R71, R15 to R72, R16 to R73, R17 to R74, R18 to R75, U9 to U20, U8 to U21
