File: right-microcode-eeprom.kicad_sch (KiCad schematic)
At the start: 20 parts, among them U37 AT28C64B, U53 74HCT04

Commit message: kicad update
Parts:
- D100: renamed from D8; footprint LED_THT:LED_D5.0mm -> 01_my_library:LED_D5.0mm
- D101: renamed from D9; footprint LED_THT:LED_D5.0mm -> 01_my_library:LED_D5.0mm
- D102: renamed from D10; footprint LED_THT:LED_D5.0mm -> 01_my_library:LED_D5.0mm
- D103: renamed from D11; footprint LED_THT:LED_D5.0mm -> 01_my_library:LED_D5.0mm
- D104: renamed from D12; footprint LED_THT:LED_D5.0mm -> 01_my_library:LED_D5.0mm
- D97: renamed from D5; footprint LED_THT:LED_D5.0mm -> 01_my_library:LED_D5.0mm
- D98: renamed from D6; footprint LED_THT:LED_D5.0mm -> 01_my_library:LED_D5.0mm
- D99: renamed from D7; footprint LED_THT:LED_D5.0mm -> 01_my_library:LED_D5.0mm
- renumbered C4 to C64, C1 to C65, R11 to R141, R12 to R142, R13 to R143, R14 to R144, R15 to R145, R16 to R146, R17 to R147, R18 to R148, U53 to U50, U37 to U51
