File: stack.kicad_sch (KiCad schematic)
At the start: 24 parts, among them U43 74HCT193, U46 74HCT193, U56 74HCT00, U7 74HCT245

Commit message: kicad update
Parts:
- D115: renamed from D5; footprint LED_THT:LED_D5.0mm -> 01_my_library:LED_D5.0mm
- D116: renamed from D6; footprint LED_THT:LED_D5.0mm -> 01_my_library:LED_D5.0mm
- D117: renamed from D7; footprint LED_THT:LED_D5.0mm -> 01_my_library:LED_D5.0mm
- D118: renamed from D8; footprint LED_THT:LED_D5.0mm -> 01_my_library:LED_D5.0mm
- D119: renamed from D9; footprint LED_THT:LED_D5.0mm -> 01_my_library:LED_D5.0mm
- D120: renamed from D10; footprint LED_THT:LED_D5.0mm -> 01_my_library:LED_D5.0mm
- D121: renamed from D11; footprint LED_THT:LED_D5.0mm -> 01_my_library:LED_D5.0mm
- D122: renamed from D12; footprint LED_THT:LED_D5.0mm -> 01_my_library:LED_D5.0mm
- renumbered C1 to C79, C1 to C80, C1 to C81, C1 to C82, R11 to R159, R12 to R160, R13 to R161, R14 to R162, R15 to R163, R16 to R164, R17 to R165, R18 to R166, U56 to U58, U7 to U63, U46 to U64, U43 to U65
